File: hw/FOCDriver.brd (EAGLE design)
At the start: 85.1 x 61 mm, 85 parts, among them U1 IX4428N, U2 IX4428N, U3 IX4428N, U4 IRF9389TRPBF, U5 IRF9389TRPBF, U6 IRF9389TRPBF, U7 LM27313XMF, U8 MCP6024T-I, U9 TLV3201AIDBVR

Commit message: layout pcb elements
Parts:
- added JP1: (no value), jumper:JP6Q
- added LED1, LED2, LED3, LED4, LED5, LED6, LED7: (no value), led:SML0805
- added R45: 1.5K 1%, resistor:R0805
- added R46: 30K 1%, resistor:R0805
- added R47: 10K 1%, resistor:R0805
- added R48: 1M 1%, resistor:R0805
- added R49, R50: 10K, resistor:R0805
- added R51: 300R 1%, resistor:R0805
- C10: value 0.1uF -> 4.7uF
- C11: value 4.7uF -> 0.1uF
- C14, C25: value 56pF -> 0.1uF
- C17: value 1nF -> 56pF
- C20: value 0.1uF -> 1nF
- C21: value 33pF -> 0.1uF
- C22: value 0.1uF -> 33pF
- C26: value 0.1uF -> 56pF
- C8: value 0.1uF -> 220pF
- C9: value 220pF -> 0.1uF
- R11: value 51K -> 1K
- R12: value 13.3K -> 1K
- R13: value 118K -> 51K
- R14, R15, R16, R17: value 1K 1% -> 1K
- R18: value 1K 1% -> 13.3K
- R19: value 1K 1% -> 118K
- R20: value 1K 1% -> 10K; device resistor:R0805 -> pot:CT6
- R21: value 1K 1% -> 100R
- R26, R27, R29, R30, R31: value 30K 1% -> 1K 1%
- R28: value 30K 1% -> 2.2K
- R35: value 1K 1% -> 30K 1%
- R36: value 1.5K 1% -> 30K 1%
- R38: value 10K 1% -> 30K 1%
- R39: value 1M 1% -> 30K 1%
- R40: value 10K -> 30K 1%
- R41: value 10K -> 1K 1%
- R42: value 300R 1% -> 1K 1%
- R43: value 10K -> 1K 1%; device pot:CT6 -> resistor:R0805
- R44: value 100R -> 1K 1%
- SV1: device con-lstb:MA05-1 -> con-lsta:FE06
- SV2: device con-lsta:FE09 -> con-lsta:FE08
- U1, U2, U3: device IX4428N:SOIC127P600X175-8N -> IX4428N:SO08
- U4, U5, U6: device IRF9389TRPBF:SOIC127P600X175-8N -> IRF9389TRPBF:SO08
- moved SV2 447.5 mm to (53.3, 76.2)
- moved C26 425.3 mm to (29.2, 64.8)
- moved R44 410.3 mm to (63.5, 52.1)
- moved R43 397.7 mm to (71.1, 52.1)
- moved C22 396.7 mm to (35.6, 64.8)
- moved C25 383.9 mm to (34.3, 58.4)
- moved C20 370.7 mm to (27.9, 71.1)
- moved R42 363.2 mm to (2.54, 45.7)
- moved R39 357.9 mm to (71.1, 39.4)
- moved C21 342.2 mm to (53.3, 58.4)
- moved R38 338.0 mm to (10.2, 33.0)
- moved C19 328.2 mm to (33.0, 71.1)
- moved R37 325.8 mm to (19.1, 33.0)
- moved R36 320.1 mm to (27.9, 33.0)
- moved C16 315.3 mm to (48.3, 64.8)
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Connections:
- removed net IMOTOR_BUS: C19.1, R34.2, R35.1, SV1.1
- new net IMOTORBUS: C20.1, R43.2, R44.1, SV1.1
- new net N$31: LED7.A, R28.1
- new net N$32: JP1.2, R11.2
- new net N$33: LED1.A, R11.1
- new net N$34: LED2.A, R12.1
- new net N$35: LED3.A, R14.1
- new net N$36: LED4.A, R15.1
- new net N$37: LED5.A, R16.1
- new net N$38: LED6.A, R17.1
- new net N$39: JP1.4, R12.2
- new net N$40: JP1.6, R14.2
- new net N$41: JP1.8, R15.2
- new net N$42: JP1.10, R16.2
- new net N$43: JP1.12, R17.2
- net +12V: now also C8.2, C9.1, R19.2; no longer C8.1, C9.2, R13.2
- net +3V3: now also C21.1, C23.2, C24.1, R20.E, R28.2, R45.2, R47.1, R49.2; no longer C20.1, C22.2, C23.1, R36.2, R38.1, R40.2, R43.E
- net AGND: now also C22.2, C26.2, R46.1; no longer C17.2, C25.2, R37.1
- net FAULT_MC: now also C26.1, R51.2; no longer C25.1, R42.2
- net GND: now also C14.2, C23.1, C25.2, C9.2, LED1.C, LED2.C, LED3.C, LED4.C, LED5.C, LED6.C, LED7.C, R18.1, R21.1, R50.1, SV1.6, SV2.8; no longer C22.1, C23.2, C26.2, C8.2, R12.1, R41.1, R44.1, SV1.5, SV2.9
- net IMOTORA: now also C18.1, R41.2; no longer C17.1, R32.2
- net IMOTORB: now also C19.1, R42.2; no longer C18.1, R33.2
- net N$1: now also R13.1; no longer R11.1
- net N$11: now also C15.2, R22.2, R29.1; no longer C14.2, R14.2, R20.1
- net N$12: now also C15.1, R23.2, R30.1; no longer C14.1, R15.2, R21.1
- net N$13: now also R29.2, R35.1; no longer R20.2, R26.1
- net N$14: now also C16.2, R24.2, R31.1; no longer C15.2, R16.2, R22.1
- net N$15: now also R30.2, R36.1; no longer R21.2, R27.1
- net N$16: now also R35.2, R41.1; no longer R26.2, R32.1
- net N$17: now also C16.1, R25.2, R32.1; no longer C15.1, R17.2, R23.1
- net N$18: now also C25.1, R49.1, R50.2; no longer C24.1, R40.1, R41.2
- net N$19: now also R31.2, R37.1; no longer R22.2, R28.1
- net N$2: now also R13.2; no longer R11.2
- net N$20: now also R32.2, R38.1; no longer R23.2, R29.1
- net N$21: now also R37.2, R42.1; no longer R28.2, R33.1
- net N$22: now also C17.2, R26.2, R33.1; no longer C16.2, R18.2, R24.1
- net N$23: now also C17.1, R27.2, R34.1; no longer C16.1, R19.2, R25.1
- net N$24: now also R33.2, R39.1; no longer R24.2, R30.1
- net N$25: now also R34.2, R40.1; no longer R25.2, R31.1
- net N$26: now also R39.2, R43.1; no longer R30.2, R34.1
- net N$27: now also C22.1, R44.2; no longer C21.1, R35.2
- net N$28: now also R45.1, R46.2, R48.1; no longer R36.1, R37.2, R39.1
- net N$29: now also C14.1, R20.A, R21.2; no longer C26.1, R43.A, R44.2
- net N$30: now also R47.2, R48.2, R51.1; no longer R38.2, R39.2, R42.1
- net N$4: now also C8.1, R18.2, R19.1; no longer C9.1, R12.2, R13.1
- net POT: now also R20.S, SV1.5; no longer R43.S, SV2.8
- net PWM1H1: now also JP1.1
- net PWM1H2: now also JP1.5
- net PWM1H3: now also JP1.9
- net PWM1L1: now also JP1.3
- net PWM1L2: now also JP1.7
- net PWM1L3: now also JP1.11
- net SHUNT_HIGH1: now also R23.1; no longer R15.1
- net SHUNT_HIGH2: now also R25.1; no longer R17.1
- net SHUNT_HIGHSUM: now also R22.1, R24.1, R27.1; no longer R14.1, R16.1, R19.1
- net SHUNT_LOWSUM: now also R26.1; no longer R18.1
- net VREF: now also R36.2, R38.2, R40.2; no longer R27.2, R29.2, R31.2
Routing:
- net +12V: track 266.1 -> 0.00 mm, vias 7 -> 0
- net GND: track 249.7 -> 0.00 mm, vias 1 -> 0
- net AGND: track 91.7 -> 0.00 mm, vias 3 -> 0
- net SHUNT_HIGHSUM: track 78.0 -> 0.00 mm, vias 2 -> 0
- net M2: track 37.5 -> 0.00 mm, vias 1 -> 0
- net N$1: track 37.0 -> 0.00 mm
- net M3: track 30.4 -> 0.00 mm, vias 1 -> 0
- net M1: track 28.9 -> 0.00 mm, vias 1 -> 0
- net PWM1L3: track 18.3 -> 0.00 mm
- net PWM1H1: track 17.9 -> 0.00 mm, vias 1 -> 0
- net N$4: track 14.9 -> 0.00 mm
- net N$12: track 13.6 -> 0.00 mm
- net N$5: track 12.3 -> 0.00 mm
- net PWM1L2: track 11.7 -> 0.00 mm
- net PWM1H3: track 9.05 -> 0.00 mm
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- removed copper zone on layer 1, net +12V
- removed copper zone on layer 1, net AGND
- removed copper zone on layer 16, net AGND
- removed copper zone on layer 16, net GND
Other:
- board size 85.1 x 61 mm -> 99.1 x 80 mm
- board text removed: "+"
- board text removed: "-"
- board text removed: "3V3"
- board text removed: "GND"
- board text removed: "H1"
- board text removed: "H2"
- board text removed: "H3"
- board text removed: "L1"
- board text removed: "L2"
- board text removed: "L3"
- board text removed: "M1_ADC"
- board text removed: "M2_ADC"
- board text removed: "M3_ADC"
- board text removed: "MOTORCUR"

Commit message: auto layout
Parts:
- R10: value 0 -> 1K
- R14: value 1K -> 0
- R7, R8, R9: device resistor:R0805 -> resistor:R2512
- moved R13 95.1 mm to (88.9, 11.4), turned to 180 degrees
- moved LED7 93.0 mm to (30.5, 3.17), turned to 90 degrees
- moved LED5 93.0 mm to (25.4, 3.17), turned to 90 degrees
- moved R14 92.0 mm to (78.7, 11.4)
- moved LED6 88.6 mm to (27.9, 3.17), turned to 90 degrees
- moved C10 86.0 mm to (78.7, 7.62)
- moved R15 80.8 mm to (22.9, 8.26), turned to 90 degrees
- moved C3 78.5 mm to (73.7, 21.6), turned to 90 degrees
- moved R38 77.3 mm to (77.5, 71.1), turned to 270 degrees
- moved R16 75.6 mm to (25.4, 8.26), turned to 90 degrees
- moved LED3 73.7 mm to (20.3, 3.17), turned to 90 degrees
- moved LED1 73.4 mm to (15.2, 3.17), turned to 90 degrees
- moved LED2 73.0 mm to (17.8, 3.17), turned to 90 degrees
- moved LED4 71.2 mm to (22.9, 3.17), turned to 90 degrees
- moved R17 71.0 mm to (27.9, 8.26), turned to 90 degrees
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Connections:
- removed net SHUNT_LOWSUM: R10.1, R26.1
- net +3V3: now also C21.2, C24.2, R47.2, SV2.2; no longer C21.1, C24.1, R47.1, SV2.1
- net AGND: now also C1.1, C10.2, C11.2, C12.-, C13.2, C2.1, C21.1, C22.1, C3.1, C4.1, C5.1, C6.1, C7.2, C9.2, R14.1, R18.1, R26.1, R46.2, R9.2, U1.3, U2.3, U3.3, U7.2, X1.2; no longer C21.2, C22.2, R10.2, R46.1, R9.1
- net FAULT_MC: now also SV1.5; no longer SV1.4
- net GND: now also C24.1, R14.2, SV2.1; no longer C1.1, C10.2, C11.2, C12.-, C13.2, C2.1, C24.2, C3.1, C4.1, C5.1, C6.1, C7.2, C9.2, R18.1, SV2.8, U1.3, U2.3, U3.3, U7.2, X1.2
- net IMOTORBUS: now also SV1.4; no longer SV1.1
- net N$19: now also R37.2; no longer R37.1
- net N$21: now also R37.1; no longer R37.2
- net N$24: now also R39.2; no longer R39.1
- net N$26: now also R39.1; no longer R39.2
- net N$27: now also C22.2; no longer C22.1
- net N$28: now also R46.1; no longer R46.2
- net N$30: now also R47.1; no longer R47.2
- net N$32: now also JP1.1, R10.2; no longer JP1.2, R11.2
- net N$33: now also R10.1; no longer R11.1
- net N$34: now also R11.1; no longer R12.1
- net N$35: now also R12.1; no longer R14.1
- net N$39: now also JP1.3, R11.2; no longer JP1.4, R12.2
- net N$40: now also JP1.5, R12.2; no longer JP1.6, R14.2
- net N$41: now also JP1.7; no longer JP1.8
- net N$42: now also JP1.9; no longer JP1.10
- net N$43: now also JP1.11; no longer JP1.12
- net POT: now also SV1.1; no longer SV1.5
- net PWM1H1: now also JP1.2, SV2.7; no longer JP1.1, SV2.3
- net PWM1H2: now also JP1.6; no longer JP1.5
- net PWM1H3: now also JP1.10, SV2.3; no longer JP1.9, SV2.7
- net PWM1L1: now also JP1.4, SV2.8; no longer JP1.3, SV2.2
- net PWM1L2: now also JP1.8, SV2.6; no longer JP1.7, SV2.4
- net PWM1L3: now also JP1.12, SV2.4; no longer JP1.11, SV2.6
- net SHUNT_HIGH1: now also R7.1; no longer R7.2
- net SHUNT_HIGH2: now also R8.1; no longer R8.2
- net SHUNT_HIGHSUM: now also R7.2, R8.2, R9.1; no longer R7.1, R8.1, R9.2
Routing:
- net AGND: track 0.00 -> 333.1 mm, vias 0 -> 8
- net GND: track 0.00 -> 294.6 mm, vias 0 -> 7
- net +3V3: track 0.00 -> 276.4 mm, vias 0 -> 5
- net +12V: track 0.00 -> 213.9 mm, vias 0 -> 3
- net SHUNT_HIGHSUM: track 0.00 -> 97.5 mm, vias 0 -> 5
- net PWM1H1: track 0.00 -> 93.2 mm
- net POT: track 0.00 -> 86.9 mm
- net N$25: track 0.00 -> 81.7 mm, vias 0 -> 2
- net IMOTORBUS: track 0.00 -> 77.9 mm, vias 0 -> 1
- net N$20: track 0.00 -> 76.3 mm, vias 0 -> 2
- net PWM1L1: track 0.00 -> 74.5 mm, vias 0 -> 1
- net PWM1L3: track 0.00 -> 71.7 mm
- net N$16: track 0.00 -> 63.6 mm, vias 0 -> 3
- net N$1: track 0.00 -> 63.2 mm, vias 0 -> 1
- net PWM1H2: track 0.00 -> 60.0 mm, vias 0 -> 1
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
Commit message: layout
Parts:
- added C27, C28: 0.1uF, resistor:C0805
- added R52: 1R, resistor:R0805
- R14: value 0 -> 0R
- moved R21 60.6 mm to (26.0, 64.1)
- moved R18 57.7 mm to (77.5, 60.3)
- moved R20 54.5 mm to (19.7, 50.2), turned to 180 degrees
- moved R19 53.9 mm to (72.4, 60.3), turned to 180 degrees
- moved C14 53.4 mm to (26.0, 59.1)
- moved C10 52.8 mm to (82.5, 60.3), turned to 180 degrees
- moved C24 52.2 mm to (26.0, 52.7), turned to 0 degrees
- moved D1 51.6 mm to (88.9, 60.3), turned to 180 degrees
- moved L1 51.2 mm to (88.9, 54.0), turned to 270 degrees
- moved U7 50.6 mm to (77.5, 54.0), turned to 270 degrees
- moved C8 44.1 mm to (72.4, 54.0), turned to 180 degrees
- moved R13 43.0 mm to (82.5, 54.0), turned to 90 degrees
- moved C12 42.8 mm to (77.5, 47.6), turned to 90 degrees
- moved C7 40.5 mm to (82.5, 47.6), turned to 270 degrees
- moved R14 36.7 mm to (72.4, 47.6)
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Connections:
- new net VDD: C21.2, C23.2, C24.2, C28.1, R45.2, R47.2, R49.2, R52.2, U8.4, U9.5
- net +3V3: now also C27.1, R52.1; no longer C21.2, C23.2, C24.2, R45.2, R47.2, R49.2, U8.4, U9.5
- net AGND: now also C23.1, C24.1, C25.2, C28.2, R14.2, R50.1, R9.1, U8.11; no longer R14.1, R9.2
- net FAULT_MC: now also SV1.4; no longer SV1.5
- net GND: now also C27.2, R14.1; no longer C23.1, C24.1, C25.2, R14.2, R50.1, U8.11
- net IMOTORA: now also SV1.3; no longer SV1.2
- net IMOTORB: now also SV1.2; no longer SV1.3
- net IMOTORBUS: now also SV1.1; no longer SV1.4
- net M1: now also X2.2; no longer X2.1
- net M2: now also X2.3; no longer X2.2
- net M3: now also X2.4; no longer X2.3
- net POT: now also SV1.5; no longer SV1.1
- net PWM1H1: now also SV2.3; no longer SV2.7
- net PWM1H3: now also SV2.7; no longer SV2.3
- net PWM1L1: now also SV2.4; no longer SV2.8
- net PWM1L3: now also SV2.8; no longer SV2.4
- net SHUNT_HIGH1: now also R7.2; no longer R7.1
- net SHUNT_HIGH2: now also R8.2; no longer R8.1
- net SHUNT_HIGHSUM: now also R7.1, R8.1, R9.2; no longer R7.2, R8.2, R9.1
Routing:
- net +3V3: track 276.4 -> 56.0 mm, vias 5 -> 2
- net VDD: track 0.00 -> 111.8 mm, vias 0 -> 6
- net GND: track 294.6 -> 192.3 mm, vias 7 -> 8
- net POT: track 86.9 -> 10.8 mm
- net PWM1H1: track 93.2 -> 24.3 mm
- net PWM1L1: track 74.5 -> 27.4 mm, vias 1 -> 0
- net N$9: track 36.9 -> 77.6 mm, vias 0 -> 2
- net N$32: track 4.77 -> 44.8 mm
- net N$1: track 63.2 -> 25.3 mm, vias 1 -> 0
- net N$39: track 4.76 -> 39.3 mm
- net PWM1L3: track 71.7 -> 39.5 mm
- net PWM1H2: track 60.0 -> 29.6 mm, vias 1 -> 0
- net N$25: track 81.7 -> 51.8 mm
- net N$40: track 4.76 -> 33.8 mm
- net N$41: track 4.77 -> 28.3 mm
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Other:
- board size 99.1 x 80 mm -> 99.1 x 68 mm

Commit message: layout
Routing:
- net GND: track 192.3 -> 281.4 mm, vias 8 -> 0
- net N$24: track 57.4 -> 100.8 mm, vias 2 -> 3
- net N$16: track 46.8 -> 89.0 mm, vias 3 -> 2
- net N$19: track 52.0 -> 83.5 mm
- net AGND: track 336.5 -> 312.9 mm, vias 7 -> 1
- net SHUNT_HIGH2: track 38.3 -> 61.4 mm
- net N$8: track 45.0 -> 67.3 mm, vias 0 -> 2
- net N$10: track 64.5 -> 44.6 mm
- net N$7: track 44.3 -> 63.7 mm
- net PWM1L2: track 45.6 -> 31.0 mm, vias 1 -> 2
- net N$26: track 13.0 -> 27.4 mm, vias 0 -> 2
- net N$29: track 17.7 -> 31.4 mm
- net N$25: track 51.8 -> 63.6 mm, vias 2 -> 3
- net N$9: track 77.6 -> 89.1 mm
- net SHUNT_HIGH1: track 49.5 -> 38.5 mm, vias 0 -> 2
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
Commit message: layout
Parts:
- C10: value 4.7uF -> 0.1uF
- C11: value 0.1uF -> 220pF
- C12: value 22uF -> 0.1uF; device resistor:E2,5-6 -> resistor:C0805
- C13: value 0.1uF -> 4.7uF
- C15: value 56pF -> 22uF; device resistor:C0805 -> resistor:E2,5-6
- C16, C17, C26: value 56pF -> 0.1uF
- C18, C19, C20: value 1nF -> 56pF
- C21, C23: value 0.1uF -> 1nF
- C22: value 33pF -> 1nF
- C25: value 0.1uF -> 33pF
- C28: value 0.1uF -> 56pF
- C7: value 10uF -> 0.1uF
- C8: value 220pF -> 10uF
- R14: value 0R -> 1R
- R15: value 1K -> 0R
- R18: value 13.3K -> 1K
- R19: value 118K -> 13.3K
- R20: value 10K -> 118K; device pot:CT6 -> resistor:R0805
- R21: value 100R -> 10K; device resistor:R0805 -> pot:CT6
- R22: value 1K 1% -> 100R
- R28: value 2.2K -> 1K 1%
- R29: value 1K 1% -> 2.2K
- R35: value 30K 1% -> 1K 1%
- R41: value 1K 1% -> 30K 1%
- R45: value 1.5K 1% -> 1K 1%
- R46: value 30K 1% -> 1.5K 1%
- R47: value 10K 1% -> 30K 1%
- R48: value 1M 1% -> 10K 1%
- R49: value 10K -> 1M 1%
- R51: value 300R 1% -> 10K
- R52: value 1R -> 300R 1%
- moved R18 77.3 mm to (12.1, 19.1)
- moved R21 68.1 mm to (93.3, 54.0)
- moved C7 66.4 mm to (17.1, 59.1), turned to 0 degrees
- moved C13 61.1 mm to (78.7, 60.3)
- moved C10 59.2 mm to (23.5, 64.1), turned to 0 degrees
- moved R14 57.7 mm to (17.1, 64.1)
- moved R29 54.8 mm to (12.1, 21.6), turned to 180 degrees
- moved C20 51.4 mm to (61.0, 10.2), turned to 270 degrees
- moved C17 51.0 mm to (87.0, 54.0), turned to 180 degrees
- moved R20 49.9 mm to (68.6, 60.3)
- moved R15 46.5 mm to (23.5, 59.1)
- moved R35 45.7 mm to (65.4, 14.0), turned to 0 degrees
- moved R28 45.1 mm to (56.5, 14.0), turned to 0 degrees
- moved C11 40.3 mm to (68.6, 54.0)
- moved R22 40.1 mm to (87.0, 60.3)
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Connections:
- net +12V: now also C11.2, C12.1, C14.1, C15.+, C16.1, R20.2; no longer C10.1, C11.1, C12.+, C8.2, C9.1, R19.2
- net +3V3: now also C7.1, R14.1, R21.E, R29.2; no longer C27.1, R20.E, R28.2, R52.1
- net AGND: now also C10.1, C12.2, C14.2, C15.-, C16.2, C21.2, C22.2, C23.2, C25.1, C26.1, C27.2, C8.2, R15.2, R19.1, R27.1, R47.2, R51.1; no longer C10.2, C11.2, C12.-, C18.2, C19.2, C20.2, C21.1, C22.1, C23.1, C25.2, C26.2, C7.2, R14.2, R18.1, R26.1, R46.2, R50.1
- net FAULT_MC: now also C28.1, R52.2; no longer C26.1, R51.2
- net GND: now also C17.2, C7.2, R15.1, R22.1; no longer C14.2, C27.2, R14.1, R21.1
- net IMOTORA: now also C21.1, R42.2; no longer C18.1, R41.2
- net IMOTORB: now also C22.1, R43.2; no longer C19.1, R42.2
- net IMOTORBUS: now also C23.1, R44.2, R45.1; no longer C20.1, R43.2, R44.1
- net N$1: now also C8.1; no longer C7.1
- net N$11: now also C18.2, R23.2, R30.1; no longer C15.2, R22.2, R29.1
- net N$12: now also C18.1, R24.2, R31.1; no longer C15.1, R23.2, R30.1
- net N$13: now also R30.2, R36.1; no longer R29.2, R35.1
- net N$14: now also C19.2, R25.2, R32.1; no longer C16.2, R24.2, R31.1
- net N$15: now also R31.2, R37.1; no longer R30.2, R36.1
- net N$16: now also R36.2, R42.1; no longer R35.2, R41.1
- net N$17: now also C19.1, R26.2, R33.1; no longer C16.1, R25.2, R32.1
- net N$18: now also C27.1, R50.1, R51.2; no longer C25.1, R49.1, R50.2
- net N$19: now also R32.2, R38.2; no longer R31.2, R37.2
- net N$20: now also R33.2, R39.1; no longer R32.2, R38.1
- net N$21: now also R38.1, R43.1; no longer R37.1, R42.1
- net N$22: now also C20.2, R27.2, R34.1; no longer C17.2, R26.2, R33.1
- net N$23: now also C20.1, R28.2, R35.1; no longer C17.1, R27.2, R34.1
- net N$24: now also R34.2, R40.2; no longer R33.2, R39.2
- net N$25: now also R35.2, R41.1; no longer R34.2, R40.1
- net N$26: now also R40.1, R44.1; no longer R39.1, R43.1
- net N$27: now also C25.2, R45.2; no longer C22.2, R44.2
- net N$28: now also R47.1, R49.1; no longer R45.1, R48.1
- net N$29: now also C17.1, R21.A, R22.2; no longer C14.1, R20.A, R21.2
- net N$30: now also R48.1, R49.2, R52.1; no longer R47.1, R48.2, R51.1
- net N$31: now also R29.1; no longer R28.1
- net N$36: now also R16.1; no longer R15.1
- net N$37: now also R17.1; no longer R16.1
- net N$38: now also R18.1; no longer R17.1
- net N$4: now also C11.1, R19.2, R20.1; no longer C8.1, R18.2, R19.1
- net N$41: now also R16.2; no longer R15.2
- net N$42: now also R17.2; no longer R16.2
- net N$43: now also R18.2; no longer R17.2
- net POT: now also R21.S; no longer R20.S
- net SHUNT_HIGH1: now also R24.1; no longer R23.1
- net SHUNT_HIGH2: now also R26.1; no longer R25.1
- net SHUNT_HIGHSUM: now also R23.1, R25.1, R28.1; no longer R22.1, R24.1, R27.1
- net VDD: now also C10.2, C26.2, C9.1, R14.2, R46.2, R48.2, R50.2; no longer C21.2, C23.2, C28.1, R45.2, R47.2, R49.2, R52.2
- net VREF: now also R37.2, R39.2, R41.2; no longer R36.2, R38.2, R40.2
Routing:
- net GND: track 281.4 -> 188.3 mm, vias 0 -> 2
- net +3V3: track 54.7 -> 144.9 mm
- net POT: track 10.8 -> 92.5 mm
- net N$9: track 89.1 -> 37.8 mm
- net AGND: track 312.9 -> 268.0 mm
- net N$16: track 89.0 -> 45.2 mm, vias 2 -> 3
- net N$24: track 100.8 -> 70.3 mm
- net N$19: track 83.5 -> 53.7 mm
- net +12V: track 208.7 -> 182.0 mm
- net VDD: track 104.6 -> 130.9 mm, vias 5 -> 2
- net N$7: track 63.7 -> 38.1 mm
- net N$8: track 67.3 -> 43.4 mm
- net SHUNT_HIGH2: track 61.4 -> 38.1 mm
- net N$29: track 31.4 -> 9.24 mm
- net PWM1H2: track 29.5 -> 47.5 mm
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
Commit message: layout
Parts:
- removed LED1, LED2, LED3, LED4, LED5, LED6, LED7: (no value), led:SML0805
- added C29: 1nF, resistor:C0805
- added FAULT, POWER, PWM1H1, PWM1H2, PWM1H3, PWM1L1, PWM1L2, PWM1L3: (no value), led:SML0805
- added R53: 1K, resistor:R0805
- C15: value 22uF -> 470uF
- moved R7 24.1 mm to (73.0, 38.1), turned to 90 degrees
- moved R8 24.1 mm to (73.0, 24.1), turned to 90 degrees
- moved R9 24.1 mm to (73.0, 10.2), turned to 270 degrees
- moved SV1 22.9 mm to (24.8, 37.5)
- moved R29 22.9 mm to (12.1, 44.5)
- moved R10 22.9 mm to (12.1, 29.2)
- moved R11 22.9 mm to (12.1, 31.8)
- moved R12 22.9 mm to (12.1, 34.3)
- moved R16 22.9 mm to (12.1, 36.8)
- moved R17 22.9 mm to (12.1, 39.4)
- moved R18 22.9 mm to (12.1, 41.9)
- moved SV2 21.3 mm to (24.8, 17.8)
- moved JP1 20.5 mm to (14.0, 15.2)
- moved R14 18.2 mm to (24.8, 47.6), turned to 270 degrees
- moved R2 10.0 mm to (37.5, 34.3)
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Connections:
- net VDD renamed AVDD
- new net N$44: FAULT.A, R53.1
- net +12V: now also C29.1
- net AGND: now also C29.2, FAULT.C
- net FAULT_MC: now also R53.2
- net GND: now also POWER.C, PWM1H1.C, PWM1H2.C, PWM1H3.C, PWM1L1.C, PWM1L2.C, PWM1L3.C; no longer LED1.C, LED2.C, LED3.C, LED4.C, LED5.C, LED6.C, LED7.C
- net N$31: now also POWER.A; no longer LED7.A
- net N$33: now also PWM1H1.A; no longer LED1.A
- net N$34: now also PWM1L1.A; no longer LED2.A
- net N$35: now also PWM1H2.A; no longer LED3.A
- net N$36: now also PWM1L2.A; no longer LED4.A
- net N$37: now also PWM1H3.A; no longer LED5.A
- net N$38: now also PWM1L3.A; no longer LED6.A
Routing:
- net AGND: track 268.0 -> 0.00 mm, vias 1 -> 0
- net GND: track 188.3 -> 0.00 mm, vias 2 -> 0
- net +12V: track 182.0 -> 0.00 mm, vias 4 -> 0
- net +3V3: track 144.9 -> 0.00 mm, vias 1 -> 0
- net AVDD: track 130.9 -> 0.00 mm, vias 2 -> 0
- net POT: track 92.5 -> 0.00 mm
- net SHUNT_HIGHSUM: track 79.9 -> 0.00 mm, vias 3 -> 0
- net N$24: track 70.3 -> 0.00 mm, vias 3 -> 0
- net N$20: track 62.3 -> 0.00 mm, vias 4 -> 0
- net N$25: track 59.4 -> 0.00 mm, vias 3 -> 0
- net N$19: track 53.7 -> 0.00 mm, vias 2 -> 0
- net IMOTORBUS: track 52.9 -> 0.00 mm, vias 2 -> 0
- net N$6: track 51.3 -> 0.00 mm
- net PWM1H2: track 47.5 -> 0.00 mm, vias 1 -> 0
- net N$32: track 47.4 -> 0.00 mm
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
Commit message: layout
Parts:
- moved R45 51.1 mm to (58.4, 17.8)
- moved C25 49.9 mm to (58.4, 21.6), turned to 180 degrees
- moved C24 47.6 mm to (47.6, 14.0)
- moved R46 46.8 mm to (47.6, 17.8), turned to 180 degrees
- moved U9 44.5 mm to (53.3, 16.5), turned to 270 degrees
- moved C23 43.9 mm to (64.1, 21.6)
- moved R44 40.7 mm to (64.1, 14.0), turned to 0 degrees
- moved R48 40.0 mm to (58.4, 14.0), turned to 180 degrees
- moved R49 35.2 mm to (53.3, 21.6), turned to 0 degrees
- moved R47 31.8 mm to (47.6, 21.6), turned to 180 degrees
- moved C10 28.9 mm to (41.9, 41.9), turned to 90 degrees
- moved FAULT 28.0 mm to (22.9, 54.0)
- moved R53 28.0 mm to (18.4, 54.0)
- moved R50 22.9 mm to (64.1, 31.1)
- moved R22 22.9 mm to (65.4, 56.5)
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Connections:
- net AGND: now also X1.1; no longer X1.2
- net N$1: now also X1.2; no longer X1.1
Routing:
- net AGND: track 0.00 -> 314.6 mm, vias 0 -> 4
- net +12V: track 0.00 -> 210.5 mm, vias 0 -> 3
- net +3V3: track 0.00 -> 130.9 mm, vias 0 -> 2
- net GND: track 0.00 -> 114.8 mm
- net AVDD: track 0.00 -> 90.3 mm, vias 0 -> 4
- net POT: track 0.00 -> 78.7 mm
- net IMOTORBUS: track 0.00 -> 78.5 mm, vias 0 -> 2
- net N$8: track 0.00 -> 63.6 mm, vias 0 -> 2
- net SHUNT_HIGHSUM: track 0.00 -> 62.9 mm, vias 0 -> 4
- net N$7: track 0.00 -> 58.6 mm, vias 0 -> 2
- net N$30: track 0.00 -> 54.7 mm, vias 0 -> 3
- net N$10: track 0.00 -> 50.2 mm, vias 0 -> 2
- net FAULT_MC: track 0.00 -> 49.8 mm, vias 0 -> 1
- net N$1: track 0.00 -> 48.4 mm
- net N$24: track 0.00 -> 46.6 mm, vias 0 -> 2
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