File: hw/FOCDriver.brd (EAGLE design)
At the start: 99.1 x 61.6 mm, 111 parts, among them Q1 BC817, Q2 BC817, Q3 BC817, Q4 BC817, Q5 BC817, Q6 BC817, U1 IRF9389TRPBF, U2 IRF9389TRPBF, U3 LM27313XMF, U4 IRF9389TRPBF, U5 LM358N, U6 LM358N, U7 SN74LVC1G17, U8 SN74LVC1G17, U9 SN74LVC1G17

Commit message: layout
Parts:
- removed U7, U8, U9: SN74LVC1G17, SN74LVC1G17:SOT23-5
- added U10, U11, U12: SN74LVC2G17, SN74LVC:SOT23-6
- R17, R2, R9: value 100 -> 1K
- moved R26 12.9 mm to (60.3, 8.26)
- moved R24 12.7 mm to (60.3, 28.9)
- moved R27 12.6 mm to (60.3, 6.03)
- moved C18 12.4 mm to (62.5, 15.2), turned to 270 degrees
- moved R25 12.3 mm to (60.3, 30.8)
- moved C17 12.0 mm to (57.5, 6.99)
- moved C16 11.5 mm to (57.5, 29.8)
- moved R32 11.1 mm to (54.6, 8.26)
- moved R30 10.9 mm to (54.6, 28.9)
- moved R33 10.7 mm to (54.6, 6.03)
- moved R31 10.5 mm to (54.6, 30.8)
- moved R35 8.26 mm to (60.3, 15.2), turned to 90 degrees
- moved R6 8.01 mm to (73.0, 40.3), turned to 90 degrees
- moved R23 6.96 mm to (66.0, 40.3)
- moved R22 6.63 mm to (66.0, 38.1)
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Connections:
- new net N$49: R1.1, R3.1, U10.4
- new net N$50: R10.1, R8.1, U11.4
- new net N$51: R16.1, R18.1, U12.4
- net +5V: now also U10.5, U11.5, U12.5; no longer U7.5, U8.5, U9.5
- net GND: now also U10.2, U11.2, U12.2; no longer U7.3, U8.3, U9.3
- net H1: now also U10.3; no longer R1.1, R3.1
- net H2: now also U11.3; no longer R10.1, R8.1
- net H3: now also U12.3; no longer R16.1, R18.1
- net L1: now also U10.1; no longer U7.2
- net L2: now also U11.1; no longer U8.2
- net L3: now also U12.1; no longer U9.2
- net N$46: now also U10.6; no longer U7.4
- net N$47: now also U11.6; no longer U8.4
- net N$48: now also U12.6; no longer U9.4
Routing:
- net AGND: track 0.00 -> 219.3 mm, vias 0 -> 1
- net GND: track 0.00 -> 157.7 mm, vias 0 -> 1
- net +12V: track 0.00 -> 126.7 mm, vias 0 -> 2
- net +5V: track 0.00 -> 110.3 mm, vias 0 -> 4
- net L1: track 0.00 -> 86.2 mm, vias 0 -> 1
- net N$9: track 0.00 -> 70.2 mm, vias 0 -> 3
- net ICOM: track 0.00 -> 66.6 mm
- net N$7: track 0.00 -> 59.6 mm, vias 0 -> 3
- net AVDD: track 0.00 -> 58.9 mm, vias 0 -> 3
- net N$6: track 0.00 -> 54.9 mm, vias 0 -> 3
- net N$3: track 0.00 -> 53.3 mm
- net N$8: track 0.00 -> 52.1 mm, vias 0 -> 3
- net VREF: track 0.00 -> 49.4 mm, vias 0 -> 2
- net N$10: track 0.00 -> 48.9 mm, vias 0 -> 2
- net L2: track 0.00 -> 41.7 mm, vias 0 -> 1
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
Commit message: layout
Parts:
- removed C9: 1nF, SparkFun-Capacitors:0805
- removed J1: (no value), SparkFun-Connectors:1X08
- removed U2, U4: IRF9389TRPBF, IRF9389TRPBF:SO08
- added C13: 47uF, rcl:E2,5-7
- added C14, C31: 0.1uF, SparkFun-Capacitors:0805
- added C2, C3, C6: 10uF, SparkFun-Capacitors:0805
- added C7: 100uF, rcl:E2,5-7
- added J3: (no value), SparkFun-Connectors:1X06
- added U7, U8, U9: AO4606, AO4606:SO08
- C10: value 4.7uF -> 0.1uF
- C11: value 470uF -> 47uF
- C19, C20: value 0.1uF -> 10uF
- R53: value 3.3K -> 1K
- U1: value IRF9389TRPBF -> SPX1117-5.0; device IRF9389TRPBF:SO08 -> SparkFun-IC-Power:SOT223
- moved U1 52.6 mm to (31.1, 55.2)
- moved R54 12.2 mm to (5.71, 48.3), turned to 0 degrees
- moved LED7 10.3 mm to (10.8, 55.2), turned to 90 degrees
- moved R53 9.52 mm to (13.3, 55.2), turned to 270 degrees
- moved C24 6.48 mm to (20.3, 42.5), turned to 180 degrees
- moved C25 5.85 mm to (20.3, 37.5), turned to 180 degrees
- moved R9 5.71 mm to (31.8, 19.1)
- moved R2 5.71 mm to (31.8, 33.0)
- moved C4 5.46 mm to (74.9, 52.1)
- moved L1 5.43 mm to (69.2, 57.8)
- moved C26 5.24 mm to (20.3, 32.4), turned to 180 degrees
- moved U3 4.84 mm to (69.2, 52.1)
- moved R42 4.02 mm to (20.3, 40.0), turned to 180 degrees
- moved R43 3.42 mm to (20.3, 34.9), turned to 180 degrees
- moved C30 3.18 mm to (19.1, 46.4)
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Connections:
- removed net N$46: R2.1, U10.6
- removed net N$47: R9.1, U11.6
- removed net N$48: R17.1, U12.6
- removed net N$49: R1.1, R3.1, U10.4
- removed net N$50: R10.1, R8.1, U11.4
- removed net N$51: R16.1, R18.1, U12.4
- new net +3V3: J2.2, R54.E
- new net H1O: R1.1, R3.1, R45.2, U10.4
- new net H2O: R10.1, R49.2, R8.1, U11.4
- new net H3O: R16.1, R18.1, R51.2, U12.4
- new net L1O: R2.1, R46.2, U10.6
- new net L2O: R50.2, R9.1, U11.6
- new net L3O: R17.1, R52.2, U12.6
- net +12V: now also C31.1, U1.3, U7.1, U8.1, U9.1; no longer C9.1, U1.1, U2.1, U4.1
- net +5V: now also C13.+, C14.1, C2.1, C3.1, C6.1, U1.2; no longer J2.1, R54.E
- net AGND: now also C13.-, C14.2, C31.2, C7.-, U1.1; no longer C9.2
- net GND: now also C2.2, C3.2, C6.2, J2.1, J3.6; no longer J1.7, J1.8, J2.2
- net H1: no longer R45.2
- net H2: no longer R49.2
- net H3: no longer R51.2
- net ICOM: now also U9.3; no longer U4.3
- net IMOTORA: now also J3.3; no longer J1.3
- net IMOTORB: now also J3.2; no longer J1.2
- net IMOTORBUS: now also J3.1; no longer J1.1
- net IU: now also U7.3; no longer U1.3
- net IV: now also U8.3; no longer U2.3
- net L1: no longer R46.2
- net L2: no longer R50.2
- net L3: no longer R52.2
- net LEDJP1: now also J3.5; no longer J1.6
- net M1: now also U7.5, U7.6, U7.7, U7.8; no longer U1.5, U1.7
- net M2: now also U8.5, U8.6, U8.7, U8.8; no longer U2.5, U2.7
- net M3: now also U9.5, U9.6, U9.7, U9.8; no longer U4.5, U4.7
- net N$1: now also C7.+
- net N$10: now also U7.2; no longer U1.2
- net N$3: now also U9.4; no longer U4.4
- net N$6: now also U9.2; no longer U4.2
- net N$7: now also U8.4; no longer U2.4
- net N$8: now also U8.2; no longer U2.2
- net N$9: now also U7.4; no longer U1.4
- net POT: now also J3.4; no longer J1.5
Routing:
- net AGND: track 219.3 -> 0.00 mm, vias 1 -> 0
- net GND: track 157.7 -> 0.00 mm, vias 1 -> 0
- net +12V: track 126.7 -> 0.00 mm, vias 2 -> 0
- net +5V: track 110.3 -> 0.00 mm, vias 4 -> 0
- net L1: track 86.2 -> 0.00 mm, vias 1 -> 0
- net N$9: track 70.2 -> 0.00 mm, vias 3 -> 0
- net ICOM: track 66.6 -> 0.00 mm
- net N$7: track 59.6 -> 0.00 mm, vias 3 -> 0
- net AVDD: track 58.9 -> 0.00 mm, vias 3 -> 0
- net N$6: track 54.9 -> 0.00 mm, vias 3 -> 0
- net N$3: track 53.3 -> 0.00 mm
- net N$8: track 52.1 -> 0.00 mm, vias 3 -> 0
- net VREF: track 49.4 -> 0.00 mm, vias 2 -> 0
- net N$10: track 48.9 -> 0.00 mm, vias 2 -> 0
- net L2: track 41.7 -> 0.00 mm, vias 1 -> 0
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Other:
- board text added: "+3V3"
- board text removed: "+5V"

Commit message: layout
Parts:
- removed C1, C12, C5: 10uF, SparkFun-Capacitors:0805
- removed C30: 0.1uF, SparkFun-Capacitors:0805
- removed C7: 100uF, rcl:E2,5-7
- removed C8: 220pF, SparkFun-Capacitors:0805
- removed L1: 10uH, resistor:L3225M
- removed LED7: 5V, led:SML0805
- removed LED8: 12V, led:SML0805
- removed R15: 118K, SparkFun-Resistors:0805
- removed R56: 10K, SparkFun-Resistors:0805
- removed U1: SPX1117-5.0, SparkFun-IC-Power:SOT223
- removed U3: LM27313XMF, LM27313XMF:SOT95P285X120-5N
- added 5VPWR: 5V, led:SML0805
- added C32, C33: 220uF/100V, rcl:E5-10,5
- added J1: (no value), SparkFun-Connectors:1X02
- added Q7: IRFR5305, transistor-power:D-PAK_TO252AA
- added U2: BA7805FP, SparkFun-IC-Power:TO-252
- C19, C2, C20, C3, C6: value 10uF -> 0.1uF
- C21, C22, C23: value 0.1uF -> 100pF
- C4: value 10uF -> 220uF/100V; device SparkFun-Capacitors:0805 -> rcl:E5-10,5
- D1: value MBR0520LT -> MM3Z18VT1G; device diode:SOD123 -> SparkFun-DiscreteSemi:SOD-323
- F1: value 16V/4.00A -> 4A/30V
- R14: value 13.3K -> 22.6K
- R34, R35, R36, R37, R38, R39, R40, R41: value 30K 1% -> 20K 1%
- R53: value 1K -> 3.3K
- R54: value (none) -> 10K
- R55: value 1K -> 5.6K
- R7: value 51K -> 100K
- moved R7 17.8 mm to (57.1, 55.9), turned to 0 degrees
- moved LED1 15.4 mm to (19.1, 21.0)
- moved LED2 15.4 mm to (19.1, 18.4)
- moved LED3 15.4 mm to (19.1, 15.9)
- moved LED4 15.4 mm to (19.1, 13.3)
- moved LED5 15.4 mm to (19.1, 10.8)
- moved LED6 15.4 mm to (19.1, 8.26)
- moved C23 15.0 mm to (57.1, 8.89), flipped to the bottom, turned to 180 degrees
- moved R41 14.7 mm to (57.1, 6.99), flipped to the bottom, turned to 0 degrees
- moved R2 12.9 mm to (36.2, 45.1), flipped to the bottom, turned to 180 degrees
- moved C21 12.1 mm to (63.2, 36.8), flipped to the bottom, turned to 90 degrees
- moved R39 11.7 mm to (65.4, 36.8), flipped to the bottom, turned to 270 degrees
- moved R45 11.6 mm to (19.1, 21.0), flipped to the bottom
- moved R46 11.6 mm to (19.1, 18.4), flipped to the bottom
- moved R49 11.6 mm to (19.1, 15.9), flipped to the bottom
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Connections:
- removed net +12V: C1.1, C10.1, C11.+, C12.1, C31.1, C5.1, C8.2, D1.C, R11.2, R15.2, R19.2, R4.2, R56.2, U1.3, U7.1, U8.1, U9.1
- removed net +3V3: J2.2, R54.E
- removed net N$29: C30.1, R54.A, R55.2
- removed net N$45: LED8.A, R56.1
- removed net N$5 (its old number): D1.A, L1.1, U3.1
- new net VCC: C10.1, C11.+, C31.1, C32.+, C33.+, C4.+, D1.C, J1.2, Q7.3, R11.2, R19.2, R4.2, R7.2, U2.1, U7.1, U8.1, U9.1
- net +5V: now also R55.2, U2.2; no longer U1.2
- net AGND: now also C32.-, C33.-, C4.-, U2.3; no longer C21.2, C22.2, C23.2, C4.2, C7.-, LED8.C, U1.1, U3.2
- net GND: now also 5VPWR.C, J2.2, R54.A; no longer C30.2, LED7.C, R55.1
- net N$1: now also J1.1, Q7.4; no longer C4.1, C7.+, L1.2, R7.1, U3.5
- net N$10: no longer C1.2
- net N$15: now also C21.2
- net N$2: now also D1.A, Q7.1, R14.2, R7.1; no longer R7.2, U3.4
- net N$20: now also C22.2
- net N$25: now also C23.2
- net N$31: now also 5VPWR.A; no longer LED7.A
- net N$4: now also R54.E, R55.1; no longer C8.1, R14.2, R15.1, U3.3
- net N$6: no longer C12.2
- net N$8: no longer C5.2
Routing:
- net AGND: track 0.00 -> 288.7 mm, vias 0 -> 4
- net VCC: track 0.00 -> 175.8 mm, vias 0 -> 1
- net GND: track 0.00 -> 155.7 mm, vias 0 -> 6
- net +5V: track 0.00 -> 119.5 mm, vias 0 -> 3
- net ICOM: track 0.00 -> 69.2 mm, vias 0 -> 2
- net AVDD: track 0.00 -> 57.6 mm, vias 0 -> 2
- net N$1: track 0.00 -> 55.2 mm
- net N$6: track 0.00 -> 54.8 mm, vias 0 -> 2
- net N$9: track 0.00 -> 51.1 mm, vias 0 -> 2
- net N$8: track 0.00 -> 48.9 mm, vias 0 -> 3
- net N$10: track 0.00 -> 48.7 mm, vias 0 -> 2
- net N$3: track 0.00 -> 48.7 mm, vias 0 -> 1
- net N$7: track 0.00 -> 48.4 mm, vias 0 -> 2
- net LEDJP1: track 0.00 -> 43.6 mm, vias 0 -> 6
- net N$26: track 0.00 -> 42.4 mm
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- added copper zone on layer 1, net AGND
- added copper zone on layer 16, net AGND
- added copper zone on layer 1, net GND
- added copper zone on layer 16, net GND
Other:
- board text added: "MA"
- board text added: "MB"
- board text added: "MC"
- board text removed: "+3V3"
- board text removed: "5 ~ 28V"
- board text removed: "M1"
- board text removed: "M2"
- board text removed: "M3"

Commit message: layout
Parts:
- moved R13 22.2 mm to (73.0, 7.62)
- moved R21 21.6 mm to (73.0, 29.5)
- moved C16 21.6 mm to (63.5, 7.94)
- moved C17 21.6 mm to (63.8, 29.5)
- moved C22 21.6 mm to (57.1, 8.89), turned to 180 degrees
- moved C23 21.6 mm to (57.1, 30.5)
- moved R24 21.6 mm to (66.4, 6.99)
- moved R25 21.6 mm to (66.4, 8.89)
- moved R26 21.6 mm to (66.7, 28.6)
- moved R27 21.6 mm to (66.7, 30.5)
- moved R30 21.6 mm to (60.6, 6.99)
- moved R31 21.6 mm to (60.6, 8.89)
- moved R32 21.6 mm to (61.0, 28.6)
- moved R33 21.6 mm to (61.0, 30.5)
- moved R37 21.6 mm to (53.3, 8.89)
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Connections:
- new net VDD: C19.1, U5.8
- net AVDD: no longer C19.1, U5.8
- net N$19: now also U6.2; no longer U5.2
- net N$20: now also U6.3; no longer U5.3
- net N$21: now also U6.1; no longer U5.1
- net N$24: now also U5.2; no longer U6.2
- net N$25: now also U5.3; no longer U6.3
- net N$26: now also U5.1; no longer U6.1
Routing:
- net AGND: track 288.7 -> 0.00 mm, vias 4 -> 0
- net VCC: track 175.8 -> 0.00 mm, vias 1 -> 0
- net GND: track 155.7 -> 0.00 mm, vias 6 -> 0
- net +5V: track 119.5 -> 0.00 mm, vias 3 -> 0
- net ICOM: track 69.2 -> 0.00 mm, vias 2 -> 0
- net AVDD: track 57.6 -> 0.00 mm, vias 2 -> 0
- net N$1: track 55.2 -> 0.00 mm
- net N$6: track 54.8 -> 0.00 mm, vias 2 -> 0
- net N$9: track 51.1 -> 0.00 mm, vias 2 -> 0
- net N$8: track 48.9 -> 0.00 mm, vias 3 -> 0
- net N$10: track 48.7 -> 0.00 mm, vias 2 -> 0
- net N$3: track 48.7 -> 0.00 mm, vias 1 -> 0
- net N$7: track 48.4 -> 0.00 mm, vias 2 -> 0
- net LEDJP1: track 43.6 -> 0.00 mm, vias 6 -> 0
- net N$26: track 42.4 -> 0.00 mm
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- removed copper zone on layer 1, net AGND
- removed copper zone on layer 16, net AGND
- removed copper zone on layer 1, net GND
- removed copper zone on layer 16, net GND
