File: hw/FOCDriver.sch (EAGLE design)
At the start: 107 parts, among them Q1 BC817, Q2 BC817, Q3 BC817, Q4 BC817, Q5 BC817, Q6 BC817, U1 SN74LVC2G17, U2 AO4606, U3 SN74LVC2G17, U4 BA7805FP, U5 AO4606, U6 SN74LVC2G17, U7 AO4606, U8 LM358N, U9 LM358N

Commit message: layout
Parts:
- removed X3: (no value), con-wago-508:W237-02P
- added J2, J4, J5, J6: (no value), SparkFun-Connectors:CONN_02
- added J7, J8: (no value), SparkFun-Connectors:CONN_06SILK_FEMALE_PTH
- added J9: (no value), SparkFun-Connectors:CONN_04
- C11: value 0.1uF -> 220uF/63V; device SparkFun-Capacitors:1.0UF-0805-25V-10% -> rcl:CPOL-USE5-10.5
- C14: value 220uF/100V -> 220uF/63V
- C2: value 220uF/100V -> 0.1uF; device rcl:CPOL-USE5-10.5 -> SparkFun-Capacitors:1.0UF-0805-25V-10%
- C3: value 0.1uF -> 47uF/50V; device SparkFun-Capacitors:1.0UF-0805-25V-10% -> rcl:CPOL-USE2.5-7
- C5: value 47uF -> 220uF/63V; device rcl:CPOL-USE2.5-7 -> rcl:CPOL-USE5-10.5
- C8: value 220uF/100V -> 47uF/50V; device rcl:CPOL-USE5-10.5 -> rcl:CPOL-USE2.5-7
- C9: value 47uF -> 0.1uF; device rcl:CPOL-USE2.5-7 -> SparkFun-Capacitors:1.0UF-0805-25V-10%
- J1, J3: device SparkFun-Connectors:CONN_06SILK_FEMALE_PTH -> SparkFun-Connectors:CONN_02
- LED1: value 5V -> ORANGE
- LED2, LED3, LED4, LED5, LED6, LED7: value (none) -> GREEN
- R12: value 180 -> 330
- R13: value 0.025R 3W 1% -> 180; device resistor:R-US_R2512 -> SparkFun-Resistors:RESISTOR0805
- R14: value 3.3K -> 0.025R 2W 1%; device SparkFun-Resistors:RESISTOR0805 -> resistor:R-US_R2512
- R22: value 0.025R 3W 1% -> 0.025R 2W 1%
- R35, R36, R37, R38, R39, R40, R41, R42: value 20K 1% -> 10K 1%
- R48, R49, R50, R51, R52, R53: value 1K -> 220
- R6: value 0.025R 3W 1% -> 0R; device resistor:R-US_R2512 -> SparkFun-Resistors:RESISTOR0805
- R7: value 0R -> 0.025R 2W 1%; device SparkFun-Resistors:RESISTOR0805 -> resistor:R-US_R2512
- U3: value SN74LVC2G17 -> BA7805FP; device SN74LVC:SN74LVC2G17 -> SparkFun-IC-Power:V_REG_78XX7812
- U4: value BA7805FP -> SN74LVC2G17; device SparkFun-IC-Power:V_REG_78XX7812 -> SN74LVC:SN74LVC2G17
- X2: device con-wago-508:W237-02P -> con-wago-500:W237-103
Connections:
- new net 3V3FROMMCU: J9.1, J9.2
- new net PWRDIV: J9.3, R35.2
- net 5V: now also C13.1, C6.1, C8.+, C9.1, R12.2, U3.OUT, U4G$1.VCC; no longer C10.1, C11.1, C4.1, C9.+, R14.2, U3G$1.VCC, U4.OUT
- net AGND: now also C10.2; no longer C13.2, Q2.E, Q4.E, Q6.E, R12.1, R21.1, R5.1
- net DGND: now also C13.2, C8.-, C9.2, J7.6, Q2.E, Q4.E, Q6.E, R13.1, R21.1, R5.1, R6.2, U3.GND, U4G$1.GND; no longer C10.2, C11.2, C9.-, J1.6, R7.2, U3G$1.GND, U4.GND
- net GND: now also C11.-, C2.2, C3.-, R6.1; no longer C2.-, C3.2, C8.-, R7.1
- net H1: now also J1.1, J8.2; no longer J3.2
- net H1O: now also J1.2
- net H2: now also J3.1, J8.6, U4G$2.A; no longer J3.4, U3G$2.A
- net H2O: now also J3.2, U4G$2.Y; no longer U3G$2.Y
- net H3: now also J5.1, J8.4; no longer J3.6
- net H3O: now also J5.2
- net ICOM: now also R14.1, R7.1; no longer R13.1, R6.1
- net IMOTORA: now also J7.3; no longer J1.3
- net IMOTORB: now also J7.1; no longer J1.1
- net IMOTORBUS: now also J7.2; no longer J1.2
- net IU: now also R7.2; no longer R6.2
- net IV: now also R14.2; no longer R13.2
- net L1: now also J2.1, J8.1; no longer J3.1
- net L1O: now also J2.2
- net L2: now also J4.1, J8.5, U4G$1.A; no longer J3.3, U3G$1.A
- net L2O: now also J4.2, U4G$1.Y; no longer U3G$1.Y
- net L3: now also J6.1, J8.3; no longer J3.5
- net L3O: now also J6.2
- net LEDJP1: now also J7.5; no longer J1.5
- net M1: now also X2-3.KL; no longer X2-1.KL
- net M2: now also X2-1.KL; no longer X3-1.KL
- net M3: now also X2-2.KL; no longer X3-2.KL
- net N$31: now also R12.1; no longer R14.1
- net N$43: now also R13.2; no longer R12.2
- net POT: now also J7.4; no longer J1.4
- net VDDA: now also C10.1, J9.4; no longer C13.1, R35.2
- net VIN: now also C11.+, C2.1, C3.+, C4.1, U3.IN; no longer C2.+, C3.1, C6.1, C8.+, U4.IN
Other:
- note added: "3.3V MCU: CONN Pin 2&3，Pin 1 3.3V come from MCU，VREF = 3.3/2 = 1.65 5.0V MCU: CONN Pin 3&4，VREF = 5.0/2 = 2.50 CAUTION:DO NOT EXCEED TARGET MCU VOLTAGE!"
- note added: "Gain: I * 0.025 * 10k / 1k = 0.25 V/A FS Current = 2.5V(1.65V) / 0.25V/A = +/-10A(+/-6.6A) F = 1/ 2 * Pi * 10k * 100pF"
- note added: "J1-J6 can switched off, and LEAVE SN74LV not installed when 5V drived MCU be engaged in."
- note added: "VREF: 5V(3.3) * 10k / 20k = 2.5V(1.65V) F = 1/ 2 * Pi * 10k||10k * 100nF"
- note removed: "Gain: I * 0.025 * 20k / 1k = 0.5 V/A FS Current = 2.5V / 0.5V/A = +/-5A F = 1/ 2 * Pi * 20k * 100pF"
- note removed: "VREF: 5V * 20k / 40k = 2.5V F = 1/ 2 * Pi * 20k||20k * 100nF"
- moved on the sheet: C10, C12, C13, C18, C4, C5, C6, C7, C8, F1, LED1, R12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

Commit message: layout
Parts:
- removed U8, U9: LM358N, Fairchild-LM358N:LM358N
- added IC1, IC2: LM258DR2G, SparkFun-IC-Amplifiers:OPAMP-DUALU
Connections:
- net AGND: now also IC1G3.P$V-, IC2G3.P$V-; no longer U8G$3.GND, U9G$3.GND
- net N$13: now also IC2G2.-IN; no longer U9G$2.-IN
- net N$15: now also IC2G2.+IN; no longer U9G$2.+IN
- net N$16: now also IC2G2.OUT; no longer U9G$2.OUT
- net N$18: now also IC1G2.+IN; no longer U8G$2.+IN
- net N$19: now also IC1G1.-IN; no longer U8G$1.-IN
- net N$20: now also IC1G1.+IN; no longer U8G$1.+IN
- net N$21: now also IC1G1.OUT; no longer U8G$1.OUT
- net N$24: now also IC2G1.-IN; no longer U9G$1.-IN
- net N$25: now also IC2G1.+IN; no longer U9G$1.+IN
- net N$26: now also IC2G1.OUT; no longer U9G$1.OUT
- net VDDA: now also IC1G3.P$V+, IC2G3.P$V+; no longer U8G$3.VCC, U9G$3.VCC
- net VREF: now also IC1G2.-IN, IC1G2.OUT; no longer U8G$2.-IN, U8G$2.OUT
Other:
- moved on the sheet: C19, C20
