File: hw/FOCDriverManual2.brd (EAGLE design)
At the start: 99.1 x 62.2 mm, 118 parts, among them Q1 BC817, Q2 BC817, Q3 BC817, Q4 BC817, Q5 BC817, Q6 BC817, U1 SN74LVC2G17, U10 LMV321SQ3T2G, U11 LMV321SQ3T2G, U2 AO4606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

Commit message: layout
Routing:
- net DGND: track 210.6 -> 0.00 mm
- net 5V: track 120.5 -> 0.00 mm, vias 1 -> 0
- net AGND: track 126.3 -> 24.8 mm, vias 2 -> 0
- net VDDA: track 107.7 -> 11.3 mm, vias 7 -> 0
- net GND: track 93.7 -> 4.81 mm, vias 2 -> 0
- net VIN: track 91.4 -> 32.3 mm
- net H1: track 58.5 -> 0.00 mm, vias 1 -> 0
- net H3: track 45.7 -> 0.00 mm, vias 1 -> 0
- net N$21: track 46.4 -> 2.54 mm, vias 2 -> 0
- net N$26: track 43.2 -> 2.54 mm, vias 2 -> 0
- net LEDJP1: track 40.6 -> 0.00 mm
- net N$16: track 42.7 -> 2.54 mm, vias 2 -> 0
- net ICOM: track 62.2 -> 22.7 mm, vias 2 -> 0
- net L1: track 38.7 -> 0.00 mm, vias 1 -> 0
- net L2: track 36.4 -> 0.00 mm
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