File: hw/dspic/dspic.brd (EAGLE design)
At the start: 60.6 x 45.7 mm, 23 parts, among them Q1 8MHz, U1 DSPIC33FJ128MC802-I/SP

Commit message: layout
Parts:
- removed S3: (no value), SparkFun-Switches:TACTILE_SWITCH_PTH_6.0MM
- removed SV2: (no value), con-lstb:MA06-1
- added J2: (no value), SparkFun-Connectors:1X02
- added R8: 0 Jump, resistor:0207/10
- added SV4, SV5: (no value), con-lstb:MA05-1
- R4, R7: value 10K -> 0 Jump
- SV1: device con-lstb:MA06-1 -> con-lstb:MA03-1
- SV3: device con-lstb:MA05-1 -> con-lstb:MA06-1
- moved R7 49.9 mm to (58.4, 24.1), turned to 90 degrees
- moved SV3 26.7 mm to (26.7, 38.1)
- moved S2 25.5 mm to (6.35, 14.0)
- moved R4 20.1 mm to (20.3, 6.35), turned to 270 degrees
- moved SV1 14.5 mm to (43.2, 38.1), turned to 180 degrees
- moved R3 5.39 mm to (53.3, 16.5)
- moved C6 4.58 mm to (36.8, 38.1)
- moved J1 4.58 mm to (55.9, 29.2)
- moved R5 4.58 mm to (6.35, 29.2)
- moved C1 4.58 mm to (33.0, 8.89)
- moved C2 4.58 mm to (40.6, 8.89)
- moved R6 4.58 mm to (6.35, 31.8)
- moved C3 4.58 mm to (44.5, 11.4)
- moved U1 4.58 mm to (31.8, 30.5)
- moved C5 4.02 mm to (14.0, 19.1)
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Connections:
- removed net N$3 (its old number): R4.2, R7.1, S3.1
- new net INT0: SV1.1, U1.16
- new net KEY: R8.1, U1.12
- new net N$4: R3.1, R4.2, R7.1, S1.1
- new net N$5: LED1.A, R4.1
- new net N$6: R5.1, R8.2
- new net U1RX: SV1.2, U1.17
- new net U1TX: SV1.3, U1.18
- net !MCLR!: now also R7.2, SV5.1; no longer LED1.A, R3.1, S1.1, SV1.1
- net +3V3: now also SV5.2; no longer S3.3, SV1.2
- net GND: now also SV4.5, SV5.3; no longer R7.2, SV1.3, SV3.5
- net H1: now also SV3.2; no longer SV2.2
- net H2: now also SV3.4; no longer SV2.4
- net H3: now also SV3.6; no longer SV2.6
- net IMOTORA: now also SV4.3, U1.4; no longer SV3.3, U1.6
- net IMOTORB: now also SV4.1; no longer SV3.1
- net IMOTORBUS: now also SV4.2; no longer SV3.2
- net L1: now also SV3.1; no longer SV2.1
- net L2: now also SV3.3; no longer SV2.3
- net L3: now also SV3.5; no longer SV2.5
- net N$10: now also J2.1, U1.6; no longer R5.1, U1.5
- net N$11: now also J2.2, U1.7; no longer R4.1, U1.4
- net PGEC: now also SV5.5; no longer SV1.5
- net PGED: now also SV5.4; no longer SV1.4
- net POT: now also SV4.4, U1.5; no longer SV3.4, U1.7
Routing:
- net N$4: track 0.00 -> 56.2 mm
- net +3V3: track 190.3 -> 153.1 mm
- net PGED: track 0.00 -> 34.3 mm
- net N$3 (its old number): track 22.4 -> 0.00 mm
- net N$6: track 0.00 -> 16.5 mm
- net N$10: track 16.5 -> 3.81 mm
- net N$3: track 27.1 -> 19.2 mm
- net POT: track 15.2 -> 7.62 mm
- net KEY: track 0.00 -> 7.62 mm
- net IMOTORA: track 15.2 -> 7.62 mm
- net !MCLR!: track 2.54 -> 8.89 mm
- net GND: track 145.6 -> 139.4 mm
- net IMOTORBUS: track 12.7 -> 7.62 mm
- net IMOTORB: track 12.7 -> 7.62 mm
- net U1TX: track 0.00 -> 3.81 mm
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Other:
- board size 60.6 x 45.7 mm -> 61.9 x 40.6 mm

Commit message: layout
Parts:
- removed SV5: (no value), con-lstb:MA05-1
- added SV2: (no value), con-lstb:MA06-1
- R5, R6: value 10K -> 0 Jump
- R7, R8: value 0 Jump -> 10K
- SV3: device con-lstb:MA06-1 -> con-lstb:MA05-1
- moved R5 52.3 mm to (58.4, 24.1), turned to 90 degrees
- moved R7 52.3 mm to (6.35, 29.2), turned to 180 degrees
- moved SV4 31.9 mm to (52.1, 31.8), turned to 90 degrees
- moved R6 26.8 mm to (33.0, 29.2), turned to 180 degrees
- moved R8 26.8 mm to (6.35, 31.8), turned to 0 degrees
- moved SV3 19.4 mm to (22.9, 19.1)
- moved S2 3.81 mm to (6.35, 10.2)
- moved R2 1.27 mm to (43.2, 19.1)
- moved C3 1.27 mm to (44.5, 12.7)
Connections:
- net !MCLR!: now also R5.2, SV4.1; no longer R7.2, SV5.1
- net +3V3: now also SV4.2; no longer SV5.2
- net GND: now also R8.2, SV3.5, SV4.3; no longer R6.2, SV4.5, SV5.3
- net H1: now also SV2.2; no longer SV3.2
- net H2: now also SV2.4; no longer SV3.4
- net H3: now also SV2.6; no longer SV3.6
- net IMOTORA: now also SV3.3; no longer SV4.3
- net IMOTORB: now also SV3.1; no longer SV4.1
- net IMOTORBUS: now also SV3.2; no longer SV4.2
- net KEY: now also R6.1; no longer R8.1
- net L1: now also SV2.1; no longer SV3.1
- net L2: now also SV2.3; no longer SV3.3
- net L3: now also SV2.5; no longer SV3.5
- net N$3: now also R7.2, R8.1; no longer R5.2, R6.1
- net N$4: now also R5.1; no longer R7.1
- net N$6: now also R6.2, R7.1; no longer R5.1, R8.2
- net PGEC: now also SV4.5; no longer SV5.5
- net PGED: now also SV4.4; no longer SV5.4
- net POT: now also SV3.4; no longer SV4.4
Routing:
- net N$3: track 19.2 -> 23.0 mm
- net N$8: track 17.9 -> 19.3 mm
- net +3V3: track 153.1 -> 154.4 mm
- net N$9: track 8.89 -> 7.62 mm

Commit message: layout
Parts:
- moved J2 3.81 mm to (27.9, 26.7)
- moved R1 3.59 mm to (40.6, 19.1)
- moved C3 2.84 mm to (43.2, 15.2)
- moved J1 2.84 mm to (54.6, 31.8)
- moved R5 2.54 mm to (58.4, 26.7)
- moved U1 2.54 mm to (31.8, 33.0)
- moved LED1 2.54 mm to (16.5, 14.0)
- moved C5 2.54 mm to (14.0, 21.6)
- moved R2 2.54 mm to (43.2, 21.6)
- moved R3 2.54 mm to (53.3, 19.1)
- moved R6 2.54 mm to (33.0, 31.8)
- moved R7 2.54 mm to (6.35, 31.8)
- moved R8 2.54 mm to (6.35, 34.3)
- moved S1 2.54 mm to (50.8, 12.7)
- moved S2 2.54 mm to (6.35, 12.7)
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Routing:
- net N$8: track 19.3 -> 23.1 mm
- net N$5: track 2.54 -> 5.08 mm
- net N$4: track 56.2 -> 58.7 mm
- net N$7: track 21.6 -> 23.9 mm
- net GND: track 139.4 -> 140.7 mm
- net +3V3: track 154.4 -> 155.7 mm
- net U1TX: track 3.81 -> 2.54 mm
- net U1RX: track 3.81 -> 2.54 mm
- net N$11: track 3.81 -> 2.54 mm
- net N$10: track 3.81 -> 2.54 mm
- net N$1: track 3.81 -> 2.54 mm
- net L3: track 3.81 -> 2.54 mm
- net L2: track 3.81 -> 2.54 mm
- net L1: track 3.81 -> 2.54 mm
- net INT0: track 3.81 -> 2.54 mm
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
Commit message: layout
Routing:
- net +3V3: track 155.7 -> 153.1 mm

Commit message: layout
Parts:
- moved R6 2.54 mm to (30.5, 31.8)
Routing:
- net N$6: track 16.5 -> 14.0 mm
- net KEY: track 7.62 -> 10.2 mm
Changed lines of the file:
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@@
 <layer number="25" name="tNames" color="7" fill="1" visible="yes" active="yes"/>
 <layer number="26" name="bNames" color="7" fill="1" visible="no" active="yes"/>
-<layer number="27" name="tValues" color="7" fill="1" visible="yes" active="yes"/>
+<layer number="27" name="tValues" color="7" fill="1" visible="no" active="yes"/>
 <layer number="28" name="bValues" color="7" fill="1" visible="no" active="yes"/>
 <layer number="29" name="tStop" color="7" fill="3" visible="no" active="yes"/>
@@
 <elements>
 <element name="C3" library="resistor" package="C025-024X044" value="0.1uF" x="43.18" y="15.24" smashed="yes" rot="R270">
-<attribute name="NAME" x="44.577" y="14.097" size="1.27" layer="25" ratio="10"/>
-<attribute name="VALUE" x="43.942" y="17.018" size="1.27" layer="27" ratio="10"/>
+<attribute name="NAME" x="44.577" y="15.748" size="1.27" layer="25" ratio="10" rot="R270"/>
+<attribute name="VALUE" x="40.513" y="17.018" size="1.27" layer="27" ratio="10" rot="R270"/>
 </element>
 <element name="C4" library="resistor" package="C025-024X044" value="0.1uF" x="16.51" y="39.37" smashed="yes" rot="R180">
-<attribute name="NAME" x="8.382" y="39.497" size="1.27" layer="25" ratio="10"/>
-<attribute name="VALUE" x="8.382" y="37.973" size="1.27" layer="27" ratio="10"/>
-</element>
-<element name="C1" library="resistor" package="C025-024X044" value="20pF" x="33.02" y="8.89" smashed="yes">
-<attribute name="NAME" x="31.242" y="10.287" size="1.27" layer="25" ratio="10"/>
-<attribute name="VALUE" x="27.432" y="6.223" size="1.27" layer="27" ratio="10"/>
-</element>
+<attribute name="NAME" x="16.002" y="40.767" size="1.27" layer="25" ratio="10"/>
+<attribute name="VALUE" x="18.288" y="42.037" size="1.27" layer="27" ratio="10" rot="R180"/>
+</element>
+<element name="C1" library="resistor" package="C025-024X044" value="20pF" x="33.02" y="8.89"/>
 <element name="C2" library="resistor" package="C025-024X044" value="20pF" x="39.37" y="8.89" smashed="yes" rot="R180">
 <attribute name="NAME" x="35.052" y="10.287" size="1.27" layer="25" ratio="10"/>
-<attribute name="VALUE" x="39.878" y="8.382" size="1.27" layer="27" ratio="10" rot="R180"/>
-</element>
-<element name="C5" library="resistor" package="C025-024X044" value="0.1uF" x="13.97" y="21.59" smashed="yes">
-<attribute name="NAME" x="12.192" y="22.987" size="1.27" layer="25" ratio="10"/>
-<attribute name="VALUE" x="9.652" y="18.923" size="1.27" layer="27" ratio="10"/>
-</element>
+<attribute name="VALUE" x="41.148" y="11.557" size="1.27" layer="27" ratio="10" rot="R180"/>
+</element>
+<element name="C5" library="resistor" package="C025-024X044" value="0.1uF" x="13.97" y="21.59"/>
 <element name="C6" library="resistor" package="C025-024X044" value="10uF" x="36.83" y="39.37" smashed="yes" rot="R180">
-<attribute name="NAME" x="35.052" y="35.052" size="1.27" layer="25" ratio="10"/>
-<attribute name="VALUE" x="38.862" y="34.798" size="1.27" layer="27" ratio="10"/>
-</element>
-<element name="LED1" library="led" package="LED3MM" value="" x="16.51" y="13.97" smashed="yes" rot="R180">
-<attribute name="NAME" x="18.415" y="15.621" size="1.27" layer="25" ratio="10"/>
-<attribute name="VALUE" x="14.605" y="15.621" size="1.27" layer="27" ratio="10" rot="R180"/>
-</element>
+<attribute name="NAME" x="36.322" y="40.767" size="1.27" layer="25" ratio="10"/>
+<attribute name="VALUE" x="38.608" y="42.037" size="1.27" layer="27" ratio="10" rot="R180"/>
+</element>
+<element name="LED1" library="led" package="LED3MM" value="" x="16.51" y="13.97" rot="R180"/>
 <element name="R2" library="resistor" package="0207/10" value="680" x="43.18" y="21.59" smashed="yes" rot="R180">
-<attribute name="NAME" x="39.497" y="24.384" size="1.27" layer="25" ratio="10"/>
-<attribute name="VALUE" x="42.1894" y="24.765" size="1.27" layer="27" ratio="10"/>
+<attribute name="NAME" x="41.402" y="24.384" size="1.27" layer="25" ratio="10"/>
+<attribute name="VALUE" x="45.4406" y="22.225" size="1.27" layer="27" ratio="10" rot="R180"/>
 </element>
 <element name="R3" library="resistor" package="0207/10" value="10K" x="53.34" y="19.05" smashed="yes" rot="R180">
@@
 <element name="R7" library="resistor" package="0207/10" value="10K" x="6.35" y="31.75" smashed="yes" rot="R180">
 <attribute name="NAME" x="3.302" y="35.814" size="1.27" layer="25" ratio="10"/>
-<attribute name="VALUE" x="-0.3556" y="28.575" size="1.27" layer="27" ratio="10"/>
+<attribute name="VALUE" x="8.6106" y="32.385" size="1.27" layer="27" ratio="10" rot="R180"/>
 </element>
 <element name="R8" library="resistor" package="0207/10" value="10K" x="6.35" y="34.29" smashed="yes">
 <attribute name="NAME" x="3.302" y="37.084" size="1.27" layer="25" ratio="10"/>
-<attribute name="VALUE" x="-0.3556" y="29.845" size="1.27" layer="27" ratio="10"/>
+<attribute name="VALUE" x="4.0894" y="33.655" size="1.27" layer="27" ratio="10"/>
 </element>
 <element name="S1" library="SparkFun-Switches" package="TACTILE_SWITCH_PTH_6.0MM" value="" x="50.8" y="12.7" rot="R180">
@@
 <attribute name="MF" value="" x="22.86" y="21.59" size="1.778" layer="27" display="off"/>
 </element>
-<element name="U1" library="Microchip-DSPIC33FJ128MC802-I_SP" package="DIP254P762X508-28" value="DSPIC33FJ128MC802-I/SP" x="31.75" y="33.02" smashed="yes" rot="R90">
+<element name="U1" library="Microchip-DSPIC33FJ128MC802-I_SP" package="DIP254P762X508-28" value="DSPIC33FJ128MC802-I/SP" x="31.75" y="33.02" rot="R90">
 <attribute name="MPN" value="DSPIC33FJ128MC802-I/SP" x="31.75" y="33.02" size="1.778" layer="27" rot="R90" display="off"/>
 <attribute name="PACKAGE" value="DIP-28" x="31.75" y="33.02" size="1.778" layer="27" rot="R90" display="off"/>
@@
 <attribute name="SUPPLIER" value="Microchip" x="31.75" y="33.02" size="1.778" layer="27" rot="R90" display="off"/>
 <attribute name="OC_FARNELL" value="1576808" x="31.75" y="33.02" size="1.778" layer="27" rot="R90" display="off"/>
-<attribute name="NAME" x="10.4648" y="28.4226" size="2.0828" layer="25" ratio="10" rot="SR0"/>
 </element>
 <element name="J1" library="SparkFun-Connectors" package="1X02" value="" x="54.61" y="31.75" rot="R90"/>
@@
 <attribute name="MF" value="" x="35.56" y="13.97" size="1.778" layer="27" rot="R180" display="off"/>
 <attribute name="NAME" x="31.75" y="16.637" size="1.27" layer="25" ratio="10"/>
+<attribute name="VALUE" x="40.64" y="17.907" size="1.27" layer="27" ratio="10" rot="R180"/>
 </element>
 <element name="R1" library="resistor" package="0207/10" value="1M" x="40.64" y="19.05" smashed="yes" rot="R180">
-<attribute name="NAME" x="38.862" y="23.114" size="1.27" layer="25" ratio="10"/>
-<attribute name="VALUE" x="41.5544" y="22.86" size="1.27" layer="27" ratio="10"/>
+<attribute name="NAME" x="40.132" y="23.114" size="1.27" layer="25" ratio="10"/>
+<attribute name="VALUE" x="42.9006" y="19.685" size="1.27" layer="27" ratio="10" rot="R180"/>
 </element>
 <element name="SV1" library="con-lstb" package="MA03-1" value="" x="43.18" y="39.37" rot="R180">
@@
 <attribute name="MPN" value="" x="43.18" y="39.37" size="1.778" layer="27" rot="R180" display="off"/>
 </element>
-<element name="R4" library="resistor" package="0207/10" value="0 Jump" x="20.32" y="6.35" smashed="yes" rot="R270">
-<attribute name="NAME" x="17.272" y="10.414" size="1.27" layer="25" ratio="10"/>
-<attribute name="VALUE" x="22.225" y="12.4206" size="1.27" layer="27" ratio="10" rot="R270"/>
-</element>
+<element name="R4" library="resistor" package="0207/10" value="0 Jump" x="20.32" y="6.35" rot="R270"/>
 <element name="R5" library="resistor" package="0207/10" value="0 Jump" x="58.42" y="26.67" smashed="yes" rot="R90">
-<attribute name="NAME" x="57.912" y="33.274" size="1.27" layer="25" ratio="10"/>
-<attribute name="VALUE" x="61.595" y="24.4094" size="1.27" layer="27" ratio="10" rot="R90"/>
-</element>
-<element name="R6" library="resistor" package="0207/10" value="0 Jump" x="33.02" y="31.75" smashed="yes" rot="R180">
-<attribute name="NAME" x="29.972" y="31.369" size="1.27" layer="25" ratio="10"/>
-<attribute name="VALUE" x="34.5694" y="31.115" size="1.27" layer="27" ratio="10"/>
+<attribute name="NAME" x="59.182" y="21.844" size="1.27" layer="25" ratio="10"/>
+<attribute name="VALUE" x="59.055" y="24.4094" size="1.27" layer="27" ratio="10" rot="R90"/>
+</element>
+<element name="R6" library="resistor" package="0207/10" value="0 Jump" x="30.48" y="31.75" smashed="yes" rot="R180">
+<attribute name="NAME" x="28.067" y="31.369" size="1.27" layer="25" ratio="10"/>
+<attribute name="VALUE" x="32.7406" y="32.385" size="1.27" layer="27" ratio="10" rot="R180"/>
 </element>
 <element name="J2" library="SparkFun-Connectors" package="1X02" value="" x="27.94" y="26.67"/>
@@
 <contactref element="U1" pad="12"/>
 <contactref element="R6" pad="1"/>
-<wire x1="38.1" y1="31.75" x2="43.18" y2="31.75" width="1.27" layer="16"/>
+<wire x1="35.56" y1="31.75" x2="43.18" y2="31.75" width="1.27" layer="16"/>
 <wire x1="43.18" y1="31.75" x2="43.18" y2="29.21" width="1.27" layer="16"/>
 </signal>
@@
 <contactref element="R7" pad="1"/>
 <contactref element="R6" pad="2"/>
-<wire x1="11.43" y1="31.75" x2="27.94" y2="31.75" width="1.27" layer="16"/>
+<wire x1="11.43" y1="31.75" x2="25.4" y2="31.75" width="1.27" layer="16"/>
 </signal>
 <signal name="N$10">

Commit message: config
Parts:
- moved S2 1.80 mm to (7.62, 11.4)
- moved C1 1.27 mm to (31.8, 8.89)
- moved J1 1.27 mm to (55.9, 31.8)
- moved SV4 1.27 mm to (53.3, 34.3)
- moved R7 1.27 mm to (7.62, 31.8)
- moved R8 1.27 mm to (7.62, 34.3)
- moved S1 1.27 mm to (50.8, 11.4)
Connections:
- removed net N$5: LED1.A, R4.1
- net GND: now also LED1.K
- net N$2: now also LED1.A, R4.1; no longer LED1.K
Routing:
- net GND: track 140.7 -> 150.9 mm
- net N$2: track 15.2 -> 22.9 mm
- net N$5: track 5.08 -> 0.00 mm
- net PGED: track 34.3 -> 33.0 mm
- net PGEC: track 6.35 -> 7.62 mm
- net !MCLR!: track 8.89 -> 7.62 mm
- net N$6: track 14.0 -> 12.7 mm
- net N$3: track 23.0 -> 22.4 mm
