File: hw/dspic/dspic.brd (EAGLE design)
At the start: 61.9 x 40.6 mm, 25 parts, among them Q1 8MHz, U1 DSPIC33FJ128MC802-I/SP

Commit message: modified pin settings
Connections:
- net IMOTORA: now also SV3.1, U1.2; no longer SV3.3, U1.4
- net IMOTORB: now also SV3.2, U1.3; no longer SV3.1, U1.2
- net IMOTORBUS: now also SV3.3, U1.4; no longer SV3.2, U1.3
Changed lines of the file:
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@@
 <wire x1="38.1" y1="19.05" x2="45.72" y2="19.05" width="1.27" layer="16"/>
 </signal>
-<signal name="IMOTORB">
+<signal name="IMOTORA">
 <contactref element="U1" pad="2"/>
 <contactref element="SV3" pad="1"/>
 <wire x1="17.78" y1="21.59" x2="17.78" y2="29.21" width="1.27" layer="16"/>
 </signal>
-<signal name="IMOTORBUS">
+<signal name="IMOTORB">
 <contactref element="U1" pad="3"/>
 <contactref element="SV3" pad="2"/>
 <wire x1="20.32" y1="21.59" x2="20.32" y2="29.21" width="1.27" layer="16"/>
 </signal>
-<signal name="IMOTORA">
+<signal name="IMOTORBUS">
 <contactref element="SV3" pad="3"/>
 <contactref element="U1" pad="4"/>
