File: hw/dspic/dspic.sch (EAGLE design)
At the start: 20 parts, among them Q1 8MH

Commit message: dspic brd
Parts:
- removed KEY1, KEY2: MOMENTARY-SWITCH-SPST-PTH-6.0MM, SparkFun-Switches:MOMENTARY-SWITCH-SPST-PTH-6.0MM
- removed U$1: DSPIC33FJ128MC802-I/SP, Microchip-DSPIC33FJ128MC802-I_SP:DSPIC33FJ128MC802-I/SP
- added J1: (no value), SparkFun-Connectors:CONN_02
- added R6, R7: 10K, resistor:R-EU_0207/10
- added S2, S3: MOMENTARY-SWITCH-SPST-PTH-6.0MM, SparkFun-Switches:MOMENTARY-SWITCH-SPST-PTH-6.0MM
- added U1: DSPIC33FJ128MC802-I/SP, Microchip-DSPIC33FJ128MC802-I_SP:DSPIC33FJ128MC802-I/SP
- C1: value 10uF -> 20pF
- C2: value 0.1uF -> 20pF
- C5: value 30pF -> 0.1uF
- C6: value 30pF -> 10uF
- Q1: value 8MH -> 8MHz; device crystal:CRYSTALHC49U70 -> crystal:CRYSTALHC49S
- R1: value 10K -> 1M
- R2: value 10K -> 680
Connections:
- removed net N$5: R2.1, U$1.PGED3/ASDA1/RP5/CN27/PMD7/RB5
- removed net N$6: R3.1, U$1.PGEC3/ASCL1/RP6/CN24/PMD6/RB6
- removed net PGC: SV1.5, U$1.PGEC1/AN3/C2IN+/RP1/CN5/RB1
- removed net PGD: SV1.4, U$1.PGED1/AN2/C2IN-/RP0/CN4/RB0
- new net N$10: R5.1, U1.PGEC1/AN3/C2IN+/RP1/CN5/RB1
- new net N$11: R4.1, U1.PGED1/AN2/C2IN-/RP0/CN4/RB0
- new net N$9: R2.2, U1.OSC2/CLKO/CN29/PMA0/RA3
- new net PGEC: SV1.5, U1.PGEC3/ASCL1/RP6/CN24/PMD6/RB6
- new net PGED: SV1.4, U1.PGED3/ASDA1/RP5/CN27/PMD7/RB5
- net !MCLR!: now also R3.1; no longer R1.1
- net +3V3: now also C4.2, J1.1, R3.2, S2.2, S3.2, U1.AVDD, U1.VDD; no longer C2.2, KEY1.2, KEY2.2, R1.2, U$1.AVDD, U$1.VDD
- net GND: now also J1.2, R6.2, R7.2, U1.AVSS, U1.VSS, U1.VSS_2; no longer R4.2, R5.2, U$1.AVSS, U$1.VSS, U$1.VSS_2
- net H1: now also U1.PWM1H1/RTCC/RP14/CN12/PMWR/RB14; no longer U$1.PWM1H1/RTCC/RP14/CN12/PMWR/RB14
- net H2: now also U1.PWM1H2/RP12/CN14/PMD0/RB12; no longer U$1.PWM1H2/RP12/CN14/PMD0/RB12
- net H3: now also U1.PGED2/TDI/PWM1H3/RP10/CN16/PMD2/RB10; no longer U$1.PGED2/TDI/PWM1H3/RP10/CN16/PMD2/RB10
- net IMOTORA: now also U1.AN4/C1IN-/RP2/CN6/RB2; no longer U$1.AN4/C1IN-/RP2/CN6/RB2
- net IMOTORB: now also U1.AN0/VREF+/CN2/RA0; no longer U$1.AN0/VREF+/CN2/RA0
- net IMOTORBUS: now also U1.AN1/VREF-/CN3/RA1; no longer U$1.AN1/VREF-/CN3/RA1
- net L1: now also U1.PWM1L1/RP15/CN11/PMCS1/RB15; no longer U$1.PWM1L1/RP15/CN11/PMCS1/RB15
- net L2: now also U1.PWM1L2/RP13/CN13/PMRD/RB13; no longer U$1.PWM1L2/RP13/CN13/PMRD/RB13
- net L3: now also U1.PGEC2/TMS/PWM1L3/RP11/CN15/PMD1/RB11; no longer U$1.PGEC2/TMS/PWM1L3/RP11/CN15/PMD1/RB11
- net N$1: now also C6.2, U1.VCAP/VDDCORE; no longer C1.2, U$1.VCAP/VDDCORE
- net N$2: now also C5.2, U1.!MCLR!; no longer C4.2, U$1.!MCLR!
- net N$3: now also R4.2, R7.1, S3.1; no longer KEY1.1, R2.2, R5.1
- net N$4: now also R5.2, R6.1, S2.1; no longer KEY2.1, R3.2, R4.1
- net N$7: now also C1.2, R1.2, U1.OSC1/CLKI/CN30/RA2; no longer C5.2, U$1.OSC1/CLKI/CN30/RA2
- net N$8: now also C2.2, R1.1, R2.1; no longer C6.2, U$1.OSC2/CLKO/CN29/PMA0/RA3
- net POT: now also U1.AN5/C1IN+/RP3/CN7/RB3; no longer U$1.AN5/C1IN+/RP3/CN7/RB3
Other:
- moved on the sheet: C1, C2, C4, C5, C6, Q1, R1, R2, R3, R4, R5, S1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

Commit message: layout
Parts:
- removed S3: MOMENTARY-SWITCH-SPST-PTH-6.0MM, SparkFun-Switches:MOMENTARY-SWITCH-SPST-PTH-6.0MM
- removed SV2: (no value), con-lstb:MA06-1
- added J2: (no value), SparkFun-Connectors:CONN_02
- added R8: 0 Jump, resistor:R-EU_0207/10
- added SV4, SV5: (no value), con-lstb:MA05-1
- R4, R7: value 10K -> 0 Jump
- SV1: device con-lstb:MA06-1 -> con-lstb:MA03-1
- SV3: device con-lstb:MA05-1 -> con-lstb:MA06-1
Connections:
- removed net N$3 (its old number): R4.2, R7.1, S3.1
- new net INT0: SV1.1, U1.INT0/RP7/CN23/PMD5/RB7
- new net KEY: R8.1, U1.SOSCO/T1CK/CN0/PMA1/RA4
- new net N$4: R3.1, R4.2, R7.1, S1.1
- new net N$5: LED1.A, R4.1
- new net N$6: R5.1, R8.2
- new net U1RX: SV1.2, U1.TCK/PWM2H1/SCL1/RP8/CN22/PMD4/RB8
- new net U1TX: SV1.3, U1.TDO/PWM2L1/SDA1/RP9/CN21/PMD3/RB9
- net !MCLR!: now also R7.2, SV5.1; no longer LED1.A, R3.1, S1.1, SV1.1
- net +3V3: now also SV5.2; no longer S3.2, SV1.2
- net GND: now also SV4.5, SV5.3; no longer R7.2, SV1.3, SV3.5
- net H1: now also SV3.2; no longer SV2.2
- net H2: now also SV3.4; no longer SV2.4
- net H3: now also SV3.6; no longer SV2.6
- net IMOTORA: now also SV4.3, U1.PGED1/AN2/C2IN-/RP0/CN4/RB0; no longer SV3.3, U1.AN4/C1IN-/RP2/CN6/RB2
- net IMOTORB: now also SV4.1; no longer SV3.1
- net IMOTORBUS: now also SV4.2; no longer SV3.2
- net L1: now also SV3.1; no longer SV2.1
- net L2: now also SV3.3; no longer SV2.3
- net L3: now also SV3.5; no longer SV2.5
- net N$10: now also J2.1, U1.AN4/C1IN-/RP2/CN6/RB2; no longer R5.1, U1.PGEC1/AN3/C2IN+/RP1/CN5/RB1
- net N$11: now also J2.2, U1.AN5/C1IN+/RP3/CN7/RB3; no longer R4.1, U1.PGED1/AN2/C2IN-/RP0/CN4/RB0
- net PGEC: now also SV5.5; no longer SV1.5
- net PGED: now also SV5.4; no longer SV1.4
- net POT: now also SV4.4, U1.PGEC1/AN3/C2IN+/RP1/CN5/RB1; no longer SV3.4, U1.AN5/C1IN+/RP3/CN7/RB3
Other:
- moved on the sheet: LED1, R3, R4, R5, R6, R7, S2

Commit message: layout
Parts:
- removed SV5: (no value), con-lstb:MA05-1
- added SV2: (no value), con-lstb:MA06-1
- R5, R6: value 10K -> 0 Jump
- R7, R8: value 0 Jump -> 10K
- SV3: device con-lstb:MA06-1 -> con-lstb:MA05-1
Connections:
- net !MCLR!: now also R5.2, SV4.1; no longer R7.2, SV5.1
- net +3V3: now also SV4.2; no longer SV5.2
- net GND: now also R8.2, SV3.5, SV4.3; no longer R6.2, SV4.5, SV5.3
- net H1: now also SV2.2; no longer SV3.2
- net H2: now also SV2.4; no longer SV3.4
- net H3: now also SV2.6; no longer SV3.6
- net IMOTORA: now also SV3.3; no longer SV4.3
- net IMOTORB: now also SV3.1; no longer SV4.1
- net IMOTORBUS: now also SV3.2; no longer SV4.2
- net KEY: now also R6.1; no longer R8.1
- net L1: now also SV2.1; no longer SV3.1
- net L2: now also SV2.3; no longer SV3.3
- net L3: now also SV2.5; no longer SV3.5
- net N$3: now also R7.2, R8.1; no longer R5.2, R6.1
- net N$4: now also R5.1; no longer R7.1
- net N$6: now also R6.2, R7.1; no longer R5.1, R8.2
- net PGEC: now also SV4.5; no longer SV5.5
- net PGED: now also SV4.4; no longer SV5.4
- net POT: now also SV3.4; no longer SV4.4
Other:
- moved on the sheet: R5, R6, R7, R8, SV4

Commit message: config
Connections:
- removed net N$5: LED1.A, R4.1
- net GND: now also LED1.C
- net N$2: now also LED1.A, R4.1; no longer LED1.C
Other:
- moved on the sheet: LED1, R3, R4, R5, S1
Changed lines of the file:
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@@
 <part name="J2" library="SparkFun-Connectors" deviceset="CONN_02" device=""/>
 <part name="SV4" library="con-lstb" deviceset="MA05-1" device=""/>
+<part name="GND11" library="supply1" deviceset="GND" device=""/>
 </parts>
 <sheets>
@@
 </plain>
 <instances>
-<instance part="R3" gate="G$1" x="40.64" y="114.3" rot="R90"/>
+<instance part="R3" gate="G$1" x="40.64" y="119.38" rot="R90"/>
 <instance part="C6" gate="G$1" x="35.56" y="53.34" rot="R90"/>
 <instance part="GND5" gate="1" x="30.48" y="40.64"/>
@@
 <instance part="GND2" gate="1" x="2.54" y="88.9" rot="R270"/>
 <instance part="+3V32" gate="G$1" x="30.48" y="93.98"/>
-<instance part="+3V33" gate="G$1" x="40.64" y="124.46"/>
+<instance part="+3V33" gate="G$1" x="40.64" y="129.54"/>
 <instance part="C5" gate="G$1" x="30.48" y="73.66" rot="R90"/>
 <instance part="GND4" gate="1" x="20.32" y="73.66" rot="R270"/>
-<instance part="S1" gate="G$1" x="60.96" y="93.98"/>
-<instance part="GND6" gate="1" x="71.12" y="91.44"/>
+<instance part="S1" gate="G$1" x="60.96" y="99.06"/>
+<instance part="GND6" gate="1" x="71.12" y="96.52"/>
 <instance part="+3V35" gate="G$1" x="170.18" y="81.28"/>
 <instance part="GND9" gate="1" x="170.18" y="71.12" rot="R270"/>
@@
 <instance part="SV3" gate="G$1" x="182.88" y="17.78" rot="R180"/>
 <instance part="GND8" gate="1" x="165.1" y="7.62"/>
-<instance part="LED1" gate="G$1" x="40.64" y="88.9"/>
+<instance part="LED1" gate="G$1" x="35.56" y="96.52"/>
 <instance part="S2" gate="G$1" x="195.58" y="93.98"/>
 <instance part="+3V36" gate="G$1" x="203.2" y="101.6"/>
@@
 <instance part="R1" gate="G$1" x="20.32" y="60.96" rot="R90"/>
 <instance part="SV1" gate="G$1" x="165.1" y="60.96" rot="R180"/>
-<instance part="R4" gate="G$1" x="40.64" y="99.06" rot="R90"/>
-<instance part="R5" gate="G$1" x="63.5" y="106.68"/>
+<instance part="R4" gate="G$1" x="40.64" y="104.14" rot="R90"/>
+<instance part="R5" gate="G$1" x="63.5" y="111.76"/>
 <instance part="R6" gate="G$1" x="152.4" y="93.98"/>
 <instance part="J2" gate="G$1" x="154.94" y="76.2" rot="R180"/>
 <instance part="SV4" gate="G$1" x="193.04" y="71.12" rot="R180"/>
+<instance part="GND11" gate="1" x="35.56" y="86.36"/>
 </instances>
 <busses>
@@
 <pinref part="S1" gate="G$1" pin="2"/>
 <pinref part="GND6" gate="1" pin="GND"/>
-<wire x1="66.04" y1="93.98" x2="71.12" y2="93.98" width="0.1524" layer="91"/>
+<wire x1="66.04" y1="99.06" x2="71.12" y2="99.06" width="0.1524" layer="91"/>
 </segment>
 <segment>
@@
 <wire x1="129.54" y1="20.32" x2="129.54" y2="17.78" width="0.1524" layer="91"/>
 </segment>
+<segment>
+<pinref part="GND11" gate="1" pin="GND"/>
+<pinref part="LED1" gate="G$1" pin="C"/>
+<wire x1="35.56" y1="88.9" x2="35.56" y2="91.44" width="0.1524" layer="91"/>
+</segment>
 </net>
 <net name="+3V3" class="0">
@@
 <pinref part="R3" gate="G$1" pin="2"/>
 <pinref part="+3V33" gate="G$1" pin="+3V3"/>
-<wire x1="40.64" y1="119.38" x2="40.64" y2="121.92" width="0.1524" layer="91"/>
+<wire x1="40.64" y1="124.46" x2="40.64" y2="127" width="0.1524" layer="91"/>
 </segment>
 <segment>
@@
 <segment>
 <pinref part="R5" gate="G$1" pin="2"/>
-<wire x1="68.58" y1="106.68" x2="73.66" y2="106.68" width="0.1524" layer="91"/>
-<label x="73.66" y="106.68" size="1.27" layer="95" xref="yes"/>
+<wire x1="68.58" y1="111.76" x2="73.66" y2="111.76" width="0.1524" layer="91"/>
+<label x="73.66" y="111.76" size="1.27" layer="95" xref="yes"/>
 </segment>
 </net>
@@
 <segment>
 <wire x1="43.18" y1="73.66" x2="40.64" y2="73.66" width="0.1524" layer="91"/>
+<pinref part="U1" gate="&gt;NAME" pin="!MCLR!"/>
+<pinref part="LED1" gate="G$1" pin="A"/>
+<pinref part="R4" gate="G$1" pin="1"/>
+<wire x1="35.56" y1="99.06" x2="40.64" y2="99.06" width="0.1524" layer="91"/>
+<wire x1="40.64" y1="73.66" x2="40.64" y2="99.06" width="0.1524" layer="91"/>
+<junction x="40.64" y="99.06"/>
 <pinref part="C5" gate="G$1" pin="2"/>
-<pinref part="LED1" gate="G$1" pin="C"/>
-<wire x1="40.64" y1="73.66" x2="35.56" y2="73.66" width="0.1524" layer="91"/>
-<wire x1="40.64" y1="83.82" x2="40.64" y2="73.66" width="0.1524" layer="91"/>
+<wire x1="35.56" y1="73.66" x2="40.64" y2="73.66" width="0.1524" layer="91"/>
 <junction x="40.64" y="73.66"/>
-<pinref part="U1" gate="&gt;NAME" pin="!MCLR!"/>
 </segment>
 </net>
@@
 </segment>
 </net>
-<net name="N$5" class="0">
-<segment>
-<pinref part="LED1" gate="G$1" pin="A"/>
-<pinref part="R4" gate="G$1" pin="1"/>
-<wire x1="40.64" y1="91.44" x2="40.64" y2="93.98" width="0.1524" layer="91"/>
-</segment>
-</net>
 <net name="N$4" class="0">
 <segment>
 <pinref part="R3" gate="G$1" pin="1"/>
 <pinref part="R4" gate="G$1" pin="2"/>
-<wire x1="40.64" y1="109.22" x2="40.64" y2="106.68" width="0.1524" layer="91"/>
+<wire x1="40.64" y1="114.3" x2="40.64" y2="111.76" width="0.1524" layer="91"/>
 <pinref part="R5" gate="G$1" pin="1"/>
-<wire x1="40.64" y1="106.68" x2="40.64" y2="104.14" width="0.1524" layer="91"/>
-<wire x1="58.42" y1="106.68" x2="53.34" y2="106.68" width="0.1524" layer="91"/>
-<junction x="40.64" y="106.68"/>
+<wire x1="40.64" y1="111.76" x2="40.64" y2="109.22" width="0.1524" layer="91"/>
+<wire x1="58.42" y1="111.76" x2="53.34" y2="111.76" width="0.1524" layer="91"/>
+<junction x="40.64" y="111.76"/>
 <pinref part="S1" gate="G$1" pin="1"/>
-<wire x1="53.34" y1="106.68" x2="40.64" y2="106.68" width="0.1524" layer="91"/>
-<wire x1="55.88" y1="93.98" x2="53.34" y2="93.98" width="0.1524" layer="91"/>
-<wire x1="53.34" y1="93.98" x2="53.34" y2="106.68" width="0.1524" layer="91"/>
-<junction x="53.34" y="106.68"/>
-</segment>
-</net>
+<wire x1="53.34" y1="111.76" x2="40.64" y2="111.76" width="0.1524" layer="91"/>
+<wire x1="55.88" y1="99.06" x2="53.34" y2="99.06" width="0.1524" layer="91"/>
+<wire x1="53.34" y1="99.06" x2="53.34" y2="111.76" width="0.1524" layer="91"/>
+<junction x="53.34" y="111.76"/>
+</segment>
+</net>

Commit message: modified pin settings
Connections:
- net IMOTORA: now also SV3.1, U1.AN0/VREF+/CN2/RA0; no longer SV3.3, U1.PGED1/AN2/C2IN-/RP0/CN4/RB0
- net IMOTORB: now also SV3.2, U1.AN1/VREF-/CN3/RA1; no longer SV3.1, U1.AN0/VREF+/CN2/RA0
- net IMOTORBUS: now also SV3.3, U1.PGED1/AN2/C2IN-/RP0/CN4/RB0; no longer SV3.2, U1.AN1/VREF-/CN3/RA1
Changed lines of the file:
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@@
 </segment>
 </net>
-<net name="IMOTORB" class="0">
+<net name="IMOTORA" class="0">
 <segment>
 <wire x1="43.18" y1="68.58" x2="38.1" y2="68.58" width="0.1524" layer="91"/>
@@
 </segment>
 </net>
-<net name="IMOTORBUS" class="0">
+<net name="IMOTORB" class="0">
 <segment>
 <wire x1="43.18" y1="66.04" x2="38.1" y2="66.04" width="0.1524" layer="91"/>
@@
 </segment>
 </net>
-<net name="IMOTORA" class="0">
+<net name="IMOTORBUS" class="0">
 <segment>
 <pinref part="SV3" gate="G$1" pin="3"/>
